File: modules/Harduino/Harduino.kicad_pcb (KiCad board)
At the start: 2 copper layers, 40.6 x 40.6 mm, 30 parts, among them J1 2, J10 11, J11 12, J12 13, J13 A0, J14 A1, J15 A2, J16 A3, J17 A4, J18 A5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

Commit message: Connect AVR to pins
Parts:
- R1: value R -> 10k
- turned U1 to 90 degrees
Connections:
- U1 pad 1: Net-(U1-Pad1) -> Net-(J2-Pad1)
- U1 pad 10: Net-(U1-Pad10) -> Net-(J5-Pad1)
- U1 pad 11: Net-(U1-Pad11) -> Net-(J6-Pad1)
- U1 pad 12: Net-(U1-Pad12) -> Net-(J7-Pad1)
- U1 pad 13: Net-(U1-Pad13) -> Net-(J8-Pad1)
- U1 pad 14: Net-(U1-Pad14) -> Net-(J9-Pad1)
- U1 pad 15: Net-(U1-Pad15) -> Net-(J10-Pad1)
- U1 pad 16: Net-(U1-Pad16) -> Net-(J11-Pad1)
- U1 pad 17: Net-(U1-Pad17) -> Net-(J12-Pad1)
- U1 pad 2: Net-(U1-Pad2) -> Net-(J3-Pad1)
- U1 pad 23: Net-(U1-Pad23) -> Net-(J13-Pad1)
- U1 pad 24: Net-(U1-Pad24) -> Net-(J14-Pad1)
- U1 pad 25: Net-(U1-Pad25) -> Net-(J15-Pad1)
- U1 pad 26: Net-(U1-Pad26) -> Net-(J16-Pad1)
- U1 pad 27: Net-(U1-Pad27) -> Net-(J17-Pad1)
- U1 pad 28: Net-(U1-Pad28) -> Net-(J18-Pad1)
- U1 pad 32: Net-(U1-Pad32) -> Net-(J1-Pad1)
- U1 pad 9: Net-(U1-Pad9) -> Net-(J4-Pad1)

Commit message: Place AVR in PCB
Parts:
- moved C3 29.8 mm to (104.5, 88.3)
- moved R1 16.5 mm to (102.2, 77.8)
- moved C2 11.4 mm to (114.3, 88.3), turned to 180 degrees
- moved C1 9.86 mm to (110.1, 63.2)
- turned Y1 to 180 degrees
Changed lines of the file:
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@@
   )
   (module Capacitor_SMD:C_0805_2012Metric_Pad1.15x1.40mm_HandSolder (layer F.Cu)
-    (at 118.355 57.785)
+    (at 110.1 63.1825)
     (descr "Capacitor SMD 0805 (2012 Metric), square (rectangular) end terminal, IPC_7351 nominal with elongated pad for handsoldering. (Body size source: https://docs.google.com/spreadsheets/d/1BsfQQcO9C6DZCsRaXUlFlo91Tg2WpOkGARC1WS5S8t0/edit?usp=sharing), generated with kicad-footprint-generator")
     (tags "capacitor handsolder")
@@
   )
   (module Capacitor_SMD:C_0805_2012Metric_Pad1.15x1.40mm_HandSolder (layer F.Cu)
-    (at 102.87 88.265 90)
+    (at 114.3 88.265 180)
     (descr "Capacitor SMD 0805 (2012 Metric), square (rectangular) end terminal, IPC_7351 nominal with elongated pad for handsoldering. (Body size source: https://docs.google.com/spreadsheets/d/1BsfQQcO9C6DZCsRaXUlFlo91Tg2WpOkGARC1WS5S8t0/edit?usp=sharing), generated with kicad-footprint-generator")
     (tags "capacitor handsolder")
     (attr smd)
-    (fp_text reference C2 (at 0 -1.65 90) (layer F.SilkS)
-      (effects (font (size 1 1) (thickness 0.15)))
-    )
-    (fp_text value C (at 0 1.65 90) (layer F.Fab)
-      (effects (font (size 1 1) (thickness 0.15)))
-    )
-    (fp_line (start -1 0.6) (end -1 -0.6) (layer F.Fab) (width 0.1))
-    (fp_line (start -1 -0.6) (end 1 -0.6) (layer F.Fab) (width 0.1))
-    (fp_line (start 1 -0.6) (end 1 0.6) (layer F.Fab) (width 0.1))
-    (fp_line (start 1 0.6) (end -1 0.6) (layer F.Fab) (width 0.1))
-    (fp_line (start -0.261252 -0.71) (end 0.261252 -0.71) (layer F.SilkS) (width 0.12))
-    (fp_line (start -0.261252 0.71) (end 0.261252 0.71) (layer F.SilkS) (width 0.12))
-    (fp_line (start -1.85 0.95) (end -1.85 -0.95) (layer F.CrtYd) (width 0.05))
-    (fp_line (start -1.85 -0.95) (end 1.85 -0.95) (layer F.CrtYd) (width 0.05))
-    (fp_line (start 1.85 -0.95) (end 1.85 0.95) (layer F.CrtYd) (width 0.05))
-    (fp_line (start 1.85 0.95) (end -1.85 0.95) (layer F.CrtYd) (width 0.05))
-    (fp_text user %R (at 0 0 90) (layer F.Fab)
-      (effects (font (size 0.5 0.5) (thickness 0.08)))
-    )
-    (pad 1 smd roundrect (at -1.025 0 90) (size 1.15 1.4) (layers F.Cu F.Paste F.Mask) (roundrect_rratio 0.217391)
+    (fp_text reference C2 (at 0 -1.65) (layer F.SilkS)
+      (effects (font (size 1 1) (thickness 0.15)))
+    )
+    (fp_text value C (at 0 1.65) (layer F.Fab)
+      (effects (font (size 1 1) (thickness 0.15)))
+    )
+    (fp_line (start -1 0.6) (end -1 -0.6) (layer F.Fab) (width 0.1))
+    (fp_line (start -1 -0.6) (end 1 -0.6) (layer F.Fab) (width 0.1))
+    (fp_line (start 1 -0.6) (end 1 0.6) (layer F.Fab) (width 0.1))
+    (fp_line (start 1 0.6) (end -1 0.6) (layer F.Fab) (width 0.1))
+    (fp_line (start -0.261252 -0.71) (end 0.261252 -0.71) (layer F.SilkS) (width 0.12))
+    (fp_line (start -0.261252 0.71) (end 0.261252 0.71) (layer F.SilkS) (width 0.12))
+    (fp_line (start -1.85 0.95) (end -1.85 -0.95) (layer F.CrtYd) (width 0.05))
+    (fp_line (start -1.85 -0.95) (end 1.85 -0.95) (layer F.CrtYd) (width 0.05))
+    (fp_line (start 1.85 -0.95) (end 1.85 0.95) (layer F.CrtYd) (width 0.05))
+    (fp_line (start 1.85 0.95) (end -1.85 0.95) (layer F.CrtYd) (width 0.05))
+    (fp_text user %R (at 0 0) (layer F.Fab)
+      (effects (font (size 0.5 0.5) (thickness 0.08)))
+    )
+    (pad 1 smd roundrect (at -1.025 0 180) (size 1.15 1.4) (layers F.Cu F.Paste F.Mask) (roundrect_rratio 0.217391)
       (net 19 "Net-(C2-Pad1)"))
-    (pad 2 smd roundrect (at 1.025 0 90) (size 1.15 1.4) (layers F.Cu F.Paste F.Mask) (roundrect_rratio 0.217391)
+    (pad 2 smd roundrect (at 1.025 0 180) (size 1.15 1.4) (layers F.Cu F.Paste F.Mask) (roundrect_rratio 0.217391)
       (net 26 GND))
     (model ${KISYS3DMOD}/Capacitor_SMD.3dshapes/C_0805_2012Metric.wrl
@@
   )
   (module Capacitor_SMD:C_0805_2012Metric_Pad1.15x1.40mm_HandSolder (layer F.Cu)
-    (at 118.99 62.23)
+    (at 104.4575 88.265)
     (descr "Capacitor SMD 0805 (2012 Metric), square (rectangular) end terminal, IPC_7351 nominal with elongated pad for handsoldering. (Body size source: https://docs.google.com/spreadsheets/d/1BsfQQcO9C6DZCsRaXUlFlo91Tg2WpOkGARC1WS5S8t0/edit?usp=sharing), generated with kicad-footprint-generator")
     (tags "capacitor handsolder")
@@
   )
   (module Resistor_SMD:R_0805_2012Metric_Pad1.15x1.40mm_HandSolder (layer F.Cu)
-    (at 114.935 88.265 90)
+    (at 102.235 77.7875 90)
     (descr "Resistor SMD 0805 (2012 Metric), square (rectangular) end terminal, IPC_7351 nominal with elongated pad for handsoldering. (Body size source: https://docs.google.com/spreadsheets/d/1BsfQQcO9C6DZCsRaXUlFlo91Tg2WpOkGARC1WS5S8t0/edit?usp=sharing), generated with kicad-footprint-generator")
     (tags "resistor handsolder")
@@
   )
   (module Crystal:Crystal_SMD_HC49-SD_HandSoldering (layer F.Cu)
-    (at 109.22 83.82)
+    (at 109.22 83.82 180)
     (descr "SMD Crystal HC-49-SD http://cdn-reichelt.de/documents/datenblatt/B400/xxx-HC49-SMD.pdf, hand-soldering, 11.4x4.7mm^2 package")
     (tags "SMD SMT crystal hand-soldering")
@@
     (fp_arc (start -3.015 0) (end -3.015 -2.115) (angle -180) (layer F.Fab) (width 0.1))
     (fp_arc (start 3.015 0) (end 3.015 -2.115) (angle 180) (layer F.Fab) (width 0.1))
-    (pad 1 smd rect (at -5.9375 0) (size 7.875 2) (layers F.Cu F.Paste F.Mask)
+    (pad 1 smd rect (at -5.9375 0 180) (size 7.875 2) (layers F.Cu F.Paste F.Mask)
       (net 19 "Net-(C2-Pad1)"))
-    (pad 2 smd rect (at 5.9375 0) (size 7.875 2) (layers F.Cu F.Paste F.Mask)
+    (pad 2 smd rect (at 5.9375 0 180) (size 7.875 2) (layers F.Cu F.Paste F.Mask)
       (net 20 "Net-(C3-Pad1)"))
     (model ${KISYS3DMOD}/Crystal.3dshapes/Crystal_SMD_HC49-SD.wrl
