File: modules/HarduinoDIP/Harduino.kicad_pcb (KiCad board)
At the start: 2 copper layers, 40.6 x 40.6 mm, 42 parts, among them J1 2, J10 11, J11 12, J12 13, J13 A0, J14 A1, J15 A2, J16 A3, J17 A4, J18 A5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

Commit message: Harduino small fixes
Parts:
- D2: footprint LED_THT:LED_D3.0mm -> LED_SMD:LED_0805_2012Metric_Pad1.15x1.40mm_HandSolder
- moved D2 0.88 mm to (99.7, 67.1)
Changed lines of the file:
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@@
   )
   (setup
-    (last_trace_width 0.6)
+    (last_trace_width 0.25)
     (user_trace_width 0.4)
     (user_trace_width 0.6)
@@
       (net 24 "Net-(C4-Pad2)"))
   )
-  (module LED_THT:LED_D3.0mm (layer F.Cu)
-    (at 99.695 67.945 90)
-    (descr "LED, diameter 3.0mm, 2 pins")
-    (tags "LED diameter 3.0mm 2 pins")
-    (fp_text reference D2 (at 1.27 -2.96 90) (layer F.SilkS)
-      (effects (font (size 1 1) (thickness 0.15)))
-    )
-    (fp_text value LED (at 1.27 2.96 90) (layer F.Fab)
-      (effects (font (size 1 1) (thickness 0.15)))
-    )
-    (fp_arc (start 1.27 0) (end -0.23 -1.16619) (angle 284.3) (layer F.Fab) (width 0.1))
-    (fp_arc (start 1.27 0) (end -0.29 -1.235516) (angle 108.8) (layer F.SilkS) (width 0.12))
-    (fp_arc (start 1.27 0) (end -0.29 1.235516) (angle -108.8) (layer F.SilkS) (width 0.12))
-    (fp_arc (start 1.27 0) (end 0.229039 -1.08) (angle 87.9) (layer F.SilkS) (width 0.12))
-    (fp_arc (start 1.27 0) (end 0.229039 1.08) (angle -87.9) (layer F.SilkS) (width 0.12))
-    (fp_circle (center 1.27 0) (end 2.77 0) (layer F.Fab) (width 0.1))
-    (fp_line (start -0.23 -1.16619) (end -0.23 1.16619) (layer F.Fab) (width 0.1))
-    (fp_line (start -0.29 -1.236) (end -0.29 -1.08) (layer F.SilkS) (width 0.12))
-    (fp_line (start -0.29 1.08) (end -0.29 1.236) (layer F.SilkS) (width 0.12))
-    (fp_line (start -1.15 -2.25) (end -1.15 2.25) (layer F.CrtYd) (width 0.05))
-    (fp_line (start -1.15 2.25) (end 3.7 2.25) (layer F.CrtYd) (width 0.05))
-    (fp_line (start 3.7 2.25) (end 3.7 -2.25) (layer F.CrtYd) (width 0.05))
-    (fp_line (start 3.7 -2.25) (end -1.15 -2.25) (layer F.CrtYd) (width 0.05))
-    (pad 1 thru_hole rect (at 0 0 90) (size 1.8 1.8) (drill 0.9) (layers *.Cu *.Mask)
-      (net 21 GND))
-    (pad 2 thru_hole circle (at 2.54 0 90) (size 1.8 1.8) (drill 0.9) (layers *.Cu *.Mask)
-      (net 25 "Net-(D2-Pad2)"))
-    (model ${KISYS3DMOD}/LED_THT.3dshapes/LED_D3.0mm.wrl
-      (at (xyz 0 0 0))
-      (scale (xyz 1 1 1))
-      (rotate (xyz 0 0 0))
-    )
-  )
   (module Connector_PinHeader_2.54mm:PinHeader_1x01_P2.54mm_Vertical (layer F.Cu)
     (at 110.1725 90.17)
@@
       (at (xyz 0 0 0))
       (scale (xyz 1 1 1))
+      (rotate (xyz 0 0 0))
+    )
+  )
+  (module LED_SMD:LED_0805_2012Metric_Pad1.15x1.40mm_HandSolder (layer F.Cu)
+    (at 99.695 67.065 90)
+    (descr "LED SMD 0805 (2012 Metric), square (rectangular) end terminal, IPC_7351 nominal, (Body size source: https://docs.google.com/spreadsheets/d/1BsfQQcO9C6DZCsRaXUlFlo91Tg2WpOkGARC1WS5S8t0/edit?usp=sharing), generated with kicad-footprint-generator")
+    (tags "LED handsolder")
+    (attr smd)
+    (fp_text reference D2 (at 0 -1.65 90) (layer F.SilkS)
+      (effects (font (size 1 1) (thickness 0.15)))
+    )
+    (fp_text value LED (at 0 1.65 90) (layer F.Fab)
+      (effects (font (size 1 1) (thickness 0.15)))
+    )
+    (fp_line (start 1 -0.6) (end -0.7 -0.6) (layer F.Fab) (width 0.1))
+    (fp_line (start -0.7 -0.6) (end -1 -0.3) (layer F.Fab) (width 0.1))
+    (fp_line (start -1 -0.3) (end -1 0.6) (layer F.Fab) (width 0.1))
+    (fp_line (start -1 0.6) (end 1 0.6) (layer F.Fab) (width 0.1))
+    (fp_line (start 1 0.6) (end 1 -0.6) (layer F.Fab) (width 0.1))
+    (fp_line (start 1 -0.96) (end -1.86 -0.96) (layer F.SilkS) (width 0.12))
+    (fp_line (start -1.86 -0.96) (end -1.86 0.96) (layer F.SilkS) (width 0.12))
+    (fp_line (start -1.86 0.96) (end 1 0.96) (layer F.SilkS) (width 0.12))
+    (fp_line (start -1.85 0.95) (end -1.85 -0.95) (layer F.CrtYd) (width 0.05))
+    (fp_line (start -1.85 -0.95) (end 1.85 -0.95) (layer F.CrtYd) (width 0.05))
+    (fp_line (start 1.85 -0.95) (end 1.85 0.95) (layer F.CrtYd) (width 0.05))
+    (fp_line (start 1.85 0.95) (end -1.85 0.95) (layer F.CrtYd) (width 0.05))
+    (fp_text user %R (at 0 0 90) (layer F.Fab)
+      (effects (font (size 0.5 0.5) (thickness 0.08)))
+    )
+    (pad 1 smd roundrect (at -1.025 0 90) (size 1.15 1.4) (layers F.Cu F.Paste F.Mask) (roundrect_rratio 0.217391)
+      (net 21 GND))
+    (pad 2 smd roundrect (at 1.025 0 90) (size 1.15 1.4) (layers F.Cu F.Paste F.Mask) (roundrect_rratio 0.217391)
+      (net 25 "Net-(D2-Pad2)"))
+    (model ${KISYS3DMOD}/LED_SMD.3dshapes/LED_0805_2012Metric.wrl
+      (at (xyz 0 0 0))
+      (scale (xyz 1 1 1))

Commit message: Harduino small fixes
Parts:
- moved R1 1.83 mm to (106.7, 81.7)
Routing:
- net Net-(C4-Pad2): track 21.0 -> 22.9 mm
Other:
- board text added: "ATmega328"
- board text added: "ISP"
Changed lines of the file:
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@@
   (general
     (thickness 1.6)
-    (drawings 34)
-    (tracks 199)
+    (drawings 36)
+    (tracks 200)
     (zones 0)
     (modules 42)
@@
   )
   (module Resistor_SMD:R_0805_2012Metric_Pad1.15x1.40mm_HandSolder (layer F.Cu)
-    (at 106.68 83.5025 270)
+    (at 106.68 81.67 270)
     (descr "Resistor SMD 0805 (2012 Metric), square (rectangular) end terminal, IPC_7351 nominal with elongated pad for handsoldering. (Body size source: https://docs.google.com/spreadsheets/d/1BsfQQcO9C6DZCsRaXUlFlo91Tg2WpOkGARC1WS5S8t0/edit?usp=sharing), generated with kicad-footprint-generator")
     (tags "resistor handsolder")
@@
     (tags "resistor handsolder")
     (attr smd)
-    (fp_text reference R2 (at 0 1.65 270) (layer B.SilkS)
+    (fp_text reference R2 (at 2.93 -0.3175 270) (layer B.SilkS)
       (effects (font (size 1 1) (thickness 0.15)) (justify mirror))
     )
@@
     (tags "resistor handsolder")
     (attr smd)
-    (fp_text reference R3 (at 0 1.65 270) (layer B.SilkS)
+    (fp_text reference R3 (at 2.785 0 270) (layer B.SilkS)
       (effects (font (size 1 1) (thickness 0.15)) (justify mirror))
     )
@@
       (rotate (xyz 0 0 0))
     )
+  )
+  (gr_text ISP (at 99.3775 87.63) (layer F.SilkS)
+    (effects (font (size 1 1) (thickness 0.15)))
+  )
+  (gr_text ATmega328 (at 106.3625 68.2625 90) (layer F.SilkS)
+    (effects (font (size 2 2) (thickness 0.25)))
   )
   (gr_text DTR (at 110.49 88.5825) (layer B.SilkS)
@@
   (segment (start 110.1725 71.12) (end 108.2675 71.12) (width 0.6) (layer F.Cu) (net 22))
   (segment (start 108.2675 71.12) (end 106.68 72.7075) (width 0.6) (layer F.Cu) (net 22))
-  (segment (start 104.775 80.9625) (end 106.68 80.9625) (width 0.6) (layer F.Cu) (net 22))
-  (segment (start 106.68 80.9625) (end 106.68 82.4775) (width 0.6) (layer F.Cu) (net 22))
+  (segment (start 104.775 79.0575) (end 106.68 79.0575) (width 0.6) (layer F.Cu) (net 22))
   (segment (start 106.68 72.7075) (end 106.68 80.9625) (width 0.6) (layer F.Cu) (net 22))
   (segment (start 102.5525 90.17) (end 102.5525 88.265) (width 0.6) (layer F.Cu) (net 22))
@@
   (segment (start 103.1875 88.265) (end 104.775 86.6775) (width 0.6) (layer F.Cu) (net 22))
   (segment (start 104.775 86.6775) (end 104.775 80.9625) (width 0.6) (layer F.Cu) (net 22))
+  (segment (start 104.775 79.0575) (end 104.775 80.9625) (width 0.6) (layer F.Cu) (net 22))
   (segment (start 110.1725 90.17) (end 117.0125 90.17) (width 0.6) (layer B.Cu) (net 23))
   (segment (start 116.84 89.9975) (end 117.0125 90.17) (width 0.6) (layer B.Cu) (net 23))
@@
   (segment (start 107.315 86.36) (end 110.1725 86.36) (width 0.6) (layer F.Cu) (net 24))
   (segment (start 106.68 85.725) (end 107.315 86.36) (width 0.6) (layer F.Cu) (net 24))
+  (segment (start 106.68 84.5275) (end 106.68 82.695) (width 0.6) (layer F.Cu) (net 24))
   (segment (start 98.28 64.135) (end 99.695 65.55) (width 0.6) (layer F.Cu) (net 25))
   (segment (start 98.28 62.23) (end 98.28 63.99) (width 0.6) (layer F.Cu) (net 25))

Commit message: Harduino small fixes
Parts:
- moved D2 2.78 mm to (97.2, 68.2)
- moved R5 1.70 mm to (98.2, 63.5)
Routing:
- net (no net): track 0.00 -> 5.08 mm
- net GND: track 95.9 -> 94.7 mm
- net VCC: track 58.7 -> 59.6 mm
- net Net-(J9-Pad1): track 29.5 -> 28.7 mm, vias 0 -> 1
- net Net-(J12-Pad1): track 13.1 -> 13.7 mm
- net Net-(J10-Pad1): vias 0 -> 1
Other:
- board text added: "+5V"
