File: modules/HarduinoDIP/Harduino.sch (KiCad schematic (older format))
At the start: 30 parts, among them J1 2, J10 11, J11 12, J12 13, J13 A0, J14 A1, J15 A2, J16 A3, J17 A4, J18 A5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

Commit message: 'Resque ATmega'
Parts:
- U1: symbol MCU_Microchip_ATmega:ATmega328P-PU -> Harduino-rescue:ATmega328P-PU-MCU_Microchip_ATmega
Changed lines of the file:
@@
 	5050 4300 5500 4300
 $Comp
-L MCU_Microchip_ATmega:ATmega328P-PU U1
+L Harduino-rescue:ATmega328P-PU-MCU_Microchip_ATmega U1
 U 1 1 5D8FD6AF
 P 2850 4850

Commit message: HarduinoDIP in work
Parts:
- added C4: 0.1uF, Capacitor_SMD:C_0805_2012Metric_Pad1.15x1.40mm_HandSolder, symbol Device:C
- added D1: 6x6-tact-btn, CommonLibrary:6x6-tact-btn, symbol CommonLibrary:6x6-tact-btn
- added D2: LED, LED_THT:LED_D3.0mm, symbol Device:LED
- added J21: ~RESET, Connector_PinHeader_2.54mm:PinHeader_1x01_P2.54mm_Vertical, symbol Connector:Conn_01x01_Male
- added J22: RX, Connector_PinHeader_2.54mm:PinHeader_1x01_P2.54mm_Vertical, symbol Connector:Conn_01x01_Male
- added J23: TX, Connector_PinHeader_2.54mm:PinHeader_1x01_P2.54mm_Vertical, symbol Connector:Conn_01x01_Male
- added J24: Vcc, Connector_PinHeader_2.54mm:PinHeader_1x01_P2.54mm_Vertical, symbol Connector:Conn_01x01_Male
- added J25: Gnd, Connector_PinHeader_2.54mm:PinHeader_1x01_P2.54mm_Vertical, symbol Connector:Conn_01x01_Male
- added R2, R3, R4, R5: 1k, Resistor_SMD:R_0805_2012Metric_Pad1.15x1.40mm_HandSolder, symbol Device:R
Connections:
- net GND: now also D1.2, D2.1 (K), J25.1 (Pin_1), R4.2
- net VCC: now also J24.1 (Pin_1)
- net at J12.1 (Pin_1), U1.19 (PB5): now also R5.2
- net at R1.2, U1.1 (~RESET~/PC6): now also C4.2, D1.1
- net at U1.2 (PD0): now also R2.2
- net at U1.3 (PD1): now also R3.2
- new net: J22.1 (Pin_1), R2.1
- new net: J23.1 (Pin_1), R3.1
- new net: C4.1, J21.1 (Pin_1), R4.1
- new net: D2.2 (A), R5.1
Changed lines of the file:
@@
 U 1 1 5D8D12B4
 P 3850 5150
-F 0 "R1" V 3775 5000 50  0000 C CNN
+F 0 "R1" V 3800 4975 50  0000 C CNN
 F 1 "10k" V 3850 5150 50  0000 C CNN
 F 2 "Resistor_SMD:R_0805_2012Metric_Pad1.15x1.40mm_HandSolder" V 3780 5150 50  0001 C CNN
@@
 $EndComp
 Wire Wire Line
-	3450 5150 3700 5150
+	3450 5150 3650 5150
 $Comp
 L power:GND #PWR0106
@@
 	4225 2950 4600 2950
 Wire Wire Line
-	4600 2950 4600 2600
+	4600 2950 4600 2850
 Wire Wire Line
 	3450 4250 4450 4250
@@
 	1    0    0    -1
 $EndComp
+$Comp
+L Device:R R2
+U 1 1 5D962682
+P 3675 5350
+F 0 "R2" V 3625 5200 50  0000 C CNN
+F 1 "1k" V 3675 5350 50  0000 C CNN
+F 2 "Resistor_SMD:R_0805_2012Metric_Pad1.15x1.40mm_HandSolder" V 3605 5350 50  0001 C CNN
+F 3 "~" H 3675 5350 50  0001 C CNN
+	1    3675 5350
+	0    1    1    0
+$EndComp
+$Comp
+L Connector:Conn_01x01_Male J22
+U 1 1 5D963134
+P 5700 5350
+F 0 "J22" H 5700 5300 50  0000 R CNN
+F 1 "RX" H 6000 5300 50  0000 R CNN
+F 2 "Connector_PinHeader_2.54mm:PinHeader_1x01_P2.54mm_Vertical" H 5700 5350 50  0001 C CNN
+F 3 "~" H 5700 5350 50  0001 C CNN
+	1    5700 5350
+	-1   0    0    1
+$EndComp
+$Comp
+L Connector:Conn_01x01_Male J23
+U 1 1 5D968559
+P 5700 5550
+F 0 "J23" H 5700 5500 50  0000 R CNN
+F 1 "TX" H 6000 5500 50  0000 R CNN
+F 2 "Connector_PinHeader_2.54mm:PinHeader_1x01_P2.54mm_Vertical" H 5700 5550 50  0001 C CNN
+F 3 "~" H 5700 5550 50  0001 C CNN
+	1    5700 5550
+	-1   0    0    1
+$EndComp
+$Comp
+L Device:R R3
+U 1 1 5D968C8D
+P 3850 5450
+F 0 "R3" V 3800 5600 50  0000 C CNN
+F 1 "1k" V 3850 5450 50  0000 C CNN
+F 2 "Resistor_SMD:R_0805_2012Metric_Pad1.15x1.40mm_HandSolder" V 3780 5450 50  0001 C CNN
+F 3 "~" H 3850 5450 50  0001 C CNN
+	1    3850 5450
+	0    1    1    0
+$EndComp
+Wire Wire Line
+	3450 5350 3525 5350
+Wire Wire Line
+	3450 5450 3700 5450
+Wire Wire Line
+	3825 5350 5500 5350
+Wire Wire Line
+	4000 5450 5250 5450
+Wire Wire Line
+	5250 5450 5250 5550
+Wire Wire Line
+	5250 5550 5500 5550
+$Comp
+L Device:C C4
+U 1 1 5D975835
+P 4750 5200
+F 0 "C4" V 4675 5075 50  0000 C CNN
+F 1 "0.1uF" V 4675 5375 50  0000 C CNN
+F 2 "Capacitor_SMD:C_0805_2012Metric_Pad1.15x1.40mm_HandSolder" H 4788 5050 50  0001 C CNN
+F 3 "~" H 4750 5200 50  0001 C CNN
+	1    4750 5200
+	0    1    1    0
+$EndComp
+Wire Wire Line
+	3650 5150 3650 5250
+Wire Wire Line
+	3650 5250 4375 5250
+Wire Wire Line
+	4375 5250 4375 5200
+Wire Wire Line
+	4375 5200 4550 5200
+Connection ~ 3650 5150
+Wire Wire Line
+	3650 5150 3700 5150
+$Comp
+L Connector:Conn_01x01_Male J21
+U 1 1 5D979C43
+P 5700 5200
+F 0 "J21" H 5700 5150 50  0000 R CNN
+F 1 "~RESET" H 6100 5150 50  0000 R CNN
+F 2 "Connector_PinHeader_2.54mm:PinHeader_1x01_P2.54mm_Vertical" H 5700 5200 50  0001 C CNN
+F 3 "~" H 5700 5200 50  0001 C CNN
+	1    5700 5200
+	-1   0    0    1
+$EndComp
+Wire Wire Line
+	4900 5200 5000 5200
+$Comp
+L Device:R R4
+U 1 1 5D97C821
+P 5000 5675
+F 0 "R4" H 5050 5700 50  0000 L CNN
+F 1 "1k" V 5000 5600 50  0000 L CNN
+F 2 "Resistor_SMD:R_0805_2012Metric_Pad1.15x1.40mm_HandSolder" V 4930 5675 50  0001 C CNN
+F 3 "~" H 5000 5675 50  0001 C CNN
+	1    5000 5675
+	1    0    0    -1
+$EndComp
+$Comp
+L power:GND #PWR01
+U 1 1 5D97D176
+P 5000 5925
+F 0 "#PWR01" H 5000 5675 50  0001 C CNN
+F 1 "GND" H 5005 5752 50  0000 C CNN
+F 2 "" H 5000 5925 50  0001 C CNN
+F 3 "" H 5000 5925 50  0001 C CNN
+	1    5000 5925
+	1    0    0    -1
+$EndComp
+Wire Wire Line
+	5000 5825 5000 5925
+Wire Wire Line
+	5000 5525 5000 5200
+Connection ~ 5000 5200
+Wire Wire Line
+	5000 5200 5500 5200
+$Comp
+L Connector:Conn_01x01_Male J24
+U 1 1 5D982630
+P 5700 5750
+F 0 "J24" H 5700 5700 50  0000 R CNN
+F 1 "Vcc" H 6000 5700 50  0000 R CNN
+F 2 "Connector_PinHeader_2.54mm:PinHeader_1x01_P2.54mm_Vertical" H 5700 5750 50  0001 C CNN
+F 3 "~" H 5700 5750 50  0001 C CNN
+	1    5700 5750
+	-1   0    0    1
+$EndComp
+$Comp
+L Connector:Conn_01x01_Male J25
+U 1 1 5D982920
+P 5700 5900
+F 0 "J25" H 5700 5850 50  0000 R CNN
+F 1 "Gnd" H 6000 5850 50  0000 R CNN
+F 2 "Connector_PinHeader_2.54mm:PinHeader_1x01_P2.54mm_Vertical" H 5700 5900 50  0001 C CNN
+F 3 "~" H 5700 5900 50  0001 C CNN
+	1    5700 5900
+	-1   0    0    1
+$EndComp
+$Comp
+L power:GND #PWR03
+U 1 1 5D9831A2
+P 5500 5900
+F 0 "#PWR03" H 5500 5650 50  0001 C CNN
+F 1 "GND" V 5505 5772 50  0000 R CNN
+F 2 "" H 5500 5900 50  0001 C CNN
+F 3 "" H 5500 5900 50  0001 C CNN
+	1    5500 5900
+	0    1    1    0
+$EndComp
+$Comp
+L power:VCC #PWR02
+U 1 1 5D9838FF
+P 5500 5750
+F 0 "#PWR02" H 5500 5600 50  0001 C CNN
+F 1 "VCC" V 5518 5877 50  0000 L CNN
+F 2 "" H 5500 5750 50  0001 C CNN
+F 3 "" H 5500 5750 50  0001 C CNN
+	1    5500 5750
+	0    -1   -1   0
+$EndComp
+$Comp
+L CommonLibrary:6x6-tact-btn D1
+U 1 1 5D98C8A9
+P 4550 5775
+F 0 "D1" V 4504 5923 50  0000 L CNN
+F 1 "6x6-tact-btn" V 4595 5923 50  0000 L CNN
+F 2 "CommonLibrary:6x6-tact-btn" H 4550 5875 50  0001 C CNN
+F 3 "" H 4550 5875 50  0001 C CNN
+	1    4550 5775
+	0    1    1    0
+$EndComp
+Wire Wire Line
+	4550 5575 4550 5200
+Connection ~ 4550 5200
+Wire Wire Line
+	4550 5200 4600 5200
+$Comp
+L power:GND #PWR04
+U 1 1 5D9919BB
+P 4550 5975
+F 0 "#PWR04" H 4550 5725 50  0001 C CNN
+F 1 "GND" H 4555 5802 50  0000 C CNN
+F 2 "" H 4550 5975 50  0001 C CNN
+F 3 "" H 4550 5975 50  0001 C CNN
+	1    4550 5975
+	1    0    0    -1
+$EndComp
+$Comp
+L Device:LED D2
+U 1 1 5D992971
+P 5200 2850
+F 0 "D2" H 5193 2595 50  0000 C CNN
+F 1 "LED" H 5193 2686 50  0000 C CNN
+F 2 "LED_THT:LED_D3.0mm" H 5200 2850 50  0001 C CNN
+F 3 "~" H 5200 2850 50  0001 C CNN
+	1    5200 2850
+	-1   0    0    1
+$EndComp
+$Comp
+L Device:R R5
+U 1 1 5D996F21
+P 4900 2850
+F 0 "R5" V 4825 2675 50  0000 C CNN
+F 1 "1k" V 4900 2825 50  0000 C CNN
+F 2 "Resistor_SMD:R_0805_2012Metric_Pad1.15x1.40mm_HandSolder" V 4830 2850 50  0001 C CNN
+F 3 "~" H 4900 2850 50  0001 C CNN
+	1    4900 2850
+	0    1    1    0
+$EndComp
+$Comp
+L power:GND #PWR05
+U 1 1 5D99A906
+P 5350 2850
+F 0 "#PWR05" H 5350 2600 50  0001 C CNN
+F 1 "GND" V 5355 2722 50  0000 R CNN
+F 2 "" H 5350 2850 50  0001 C CNN
+F 3 "" H 5350 2850 50  0001 C CNN
+	1    5350 2850
+	0    -1   -1   0
+$EndComp
+Wire Wire Line
+	4750 2850 4600 2850
+Connection ~ 4600 2850
+Wire Wire Line
+	4600 2850 4600 2600
 $EndSCHEMATC

Commit message: Harduino small fixes
Parts:
- D2: footprint LED_THT:LED_D3.0mm -> LED_SMD:LED_0805_2012Metric_Pad1.15x1.40mm_HandSolder
Changed lines of the file:
@@
 F 0 "D2" H 5193 2595 50  0000 C CNN
 F 1 "LED" H 5193 2686 50  0000 C CNN
-F 2 "LED_THT:LED_D3.0mm" H 5200 2850 50  0001 C CNN
+F 2 "LED_SMD:LED_0805_2012Metric_Pad1.15x1.40mm_HandSolder" H 5200 2850 50  0001 C CNN
 F 3 "~" H 5200 2850 50  0001 C CNN
 	1    5200 2850

Commit message: Lost values
Parts:
- C1: value C -> 0,1uF
- C2, C3: value C -> 22pF
Changed lines of the file:
@@
 P 4925 4125
 F 0 "C2" H 5040 4171 50  0000 L CNN
-F 1 "C" H 5040 4080 50  0000 L CNN
+F 1 "22pF" H 5040 4080 50  0000 L CNN
 F 2 "Capacitor_SMD:C_0805_2012Metric_Pad1.15x1.40mm_HandSolder" H 4963 3975 50  0001 C CNN
 F 3 "~" H 4925 4125 50  0001 C CNN
@@
 P 4925 3400
 F 0 "C3" H 5040 3446 50  0000 L CNN
-F 1 "C" H 5040 3355 50  0000 L CNN
+F 1 "22pF" H 5040 3355 50  0000 L CNN
 F 2 "Capacitor_SMD:C_0805_2012Metric_Pad1.15x1.40mm_HandSolder" H 4963 3250 50  0001 C CNN
 F 3 "~" H 4925 3400 50  0001 C CNN
@@
 P 3375 3225
 F 0 "C1" H 3490 3271 50  0000 L CNN
-F 1 "C" H 3490 3180 50  0000 L CNN
+F 1 "0,1uF" H 3490 3180 50  0000 L CNN
 F 2 "Capacitor_SMD:C_0805_2012Metric_Pad1.15x1.40mm_HandSolder" H 3413 3075 50  0001 C CNN
 F 3 "~" H 3375 3225 50  0001 C CNN
