File: modules/Kbd/Kbd.kicad_pcb (KiCad board)
At the start: 2 copper layers, 40.6 x 40.6 mm, 36 parts, among them J1 2, J10 11, J11 12, J12 13, J13 A0, J14 A1, J15 A2, J16 A3, J17 A4, J18 A5, J19 Vcc, J2 3, J20 Gnd, J3 4, J4 5, J5 6, J6 7, J7 8, J8 9, J9 10

Commit message: Raw Kbd in work
Parts:
- added R1: 10k, Resistor_SMD:R_0805_2012Metric_Pad1.15x1.40mm_HandSolder, F.Cu at (99.6, 45.4)
- added R2: 10k, Resistor_SMD:R_0805_2012Metric_Pad1.15x1.40mm_HandSolder, F.Cu at (106.0, 42.5)
- added R3: 10k, Resistor_SMD:R_0805_2012Metric_Pad1.15x1.40mm_HandSolder, F.Cu at (114.2, 36.5)
- added VD1: LL4148, Diode_SMD:D_MiniMELF, B.Cu at (118.9, 56.4)
- added VD2: LL4148, Diode_SMD:D_MiniMELF, B.Cu at (119.4, 66.0)
- added VD3: LL4148, Diode_SMD:D_MiniMELF, B.Cu at (119.4, 76.7)
- added VD4: LL4148, Diode_SMD:D_MiniMELF, B.Cu at (119.1, 86.4)
- moved D10 30.5 mm to (98.7, 89.5)
- moved D3 30.5 mm to (115.3, 59.1)
- moved D7 21.9 mm to (98.7, 79.4)
- moved D1 20.3 mm to (98.7, 59.1)
- moved D11 20.3 mm to (107.0, 89.5)
- moved D8 13.1 mm to (107.0, 79.4)
- moved D5 10.2 mm to (107.0, 69.2)
- moved D6 10.2 mm to (115.3, 69.2)
- moved D9 10.2 mm to (115.3, 79.4)
- moved D12 8.25 mm to (115.3, 89.5)
- moved D2 8.25 mm to (107.0, 59.1)
- renumbered D1004 to D1, D1001 to D10, D1005 to D11, D1009 to D12, D1008 to D2, D1012 to D3, D1002 to D4, D1006 to D5, D1010 to D6, D1003 to D7, D1007 to D8, D1011 to D9
Connections:
- D1 pad 1: Net-(D1004-Pad1) -> Net-(D1-Pad1)
- D1 pad 2: Net-(D1004-Pad2) -> Net-(D1-Pad2)
- D10 pad 1: Net-(D1001-Pad1) -> Net-(D1-Pad1)
- D10 pad 2: Net-(D1001-Pad2) -> Net-(D10-Pad2)
- D11 pad 1: Net-(D1005-Pad1) -> Net-(D11-Pad1)
- D11 pad 2: Net-(D1005-Pad2) -> Net-(D10-Pad2)
- D12 pad 1: Net-(D1009-Pad1) -> Net-(D12-Pad1)
- D12 pad 2: Net-(D1009-Pad2) -> Net-(D10-Pad2)
- D2 pad 1: Net-(D1008-Pad1) -> Net-(D11-Pad1)
- D2 pad 2: Net-(D1008-Pad2) -> Net-(D1-Pad2)
- D3 pad 1: Net-(D1012-Pad1) -> Net-(D12-Pad1)
- D3 pad 2: Net-(D1012-Pad2) -> Net-(D1-Pad2)
- D4 pad 1: Net-(D1002-Pad1) -> Net-(D1-Pad1)
- D4 pad 2: Net-(D1002-Pad2) -> Net-(D4-Pad2)
- D5 pad 1: Net-(D1006-Pad1) -> Net-(D11-Pad1)
- D5 pad 2: Net-(D1006-Pad2) -> Net-(D4-Pad2)
- D6 pad 1: Net-(D1010-Pad1) -> Net-(D12-Pad1)
- D6 pad 2: Net-(D1010-Pad2) -> Net-(D4-Pad2)
- D7 pad 1: Net-(D1003-Pad1) -> Net-(D1-Pad1)
- D7 pad 2: Net-(D1003-Pad2) -> Net-(D7-Pad2)
- D8 pad 1: Net-(D1007-Pad1) -> Net-(D11-Pad1)
- D8 pad 2: Net-(D1007-Pad2) -> Net-(D7-Pad2)
- D9 pad 1: Net-(D1011-Pad1) -> Net-(D12-Pad1)
- D9 pad 2: Net-(D1011-Pad2) -> Net-(D7-Pad2)
- J13 pad 1: Net-(J13-Pad1) -> Net-(D12-Pad1)
- J14 pad 1: Net-(J14-Pad1) -> Net-(D11-Pad1)
- J15 pad 1: Net-(J15-Pad1) -> Net-(D1-Pad1)
Routing:
- net Net-(D7-Pad2): track 0.00 -> 23.7 mm
- net Net-(D1-Pad2): track 0.00 -> 23.7 mm
- net Net-(D4-Pad2): track 0.00 -> 23.1 mm
- net Net-(J6-Pad1): track 0.00 -> 16.5 mm
- net Net-(J3-Pad1): track 0.00 -> 11.9 mm
- net Net-(D12-Pad1): track 0.00 -> 11.0 mm
- net Net-(D11-Pad1): track 0.00 -> 11.0 mm
- net Net-(D1-Pad1): track 0.00 -> 11.0 mm
- net Net-(J5-Pad1): track 0.00 -> 9.45 mm
- net Net-(J4-Pad1): track 0.00 -> 5.47 mm
- net Net-(D10-Pad2): track 0.00 -> 5.27 mm

Commit message: Raw Kbd is ready
Parts:
- R1, R2, R3: moved to B.Cu
- moved R3 20.0 mm to (114.3, 56.5)
- moved R1 15.8 mm to (95.9, 60.7), turned to 270 degrees
- moved R2 15.3 mm to (109.2, 57.5), turned to 270 degrees
- moved VD1 6.38 mm to (122.6, 61.6), turned to 90 degrees
Routing:
- net Net-(D12-Pad1): track 11.0 -> 38.9 mm
- net Net-(J19-Pad1): track 0.00 -> 23.0 mm
- net Net-(D11-Pad1): track 11.0 -> 30.7 mm
- net Net-(D1-Pad1): track 11.0 -> 20.5 mm
- net Net-(J6-Pad1): track 16.5 -> 8.68 mm
- net Net-(D1-Pad2): track 23.7 -> 29.3 mm
Other:
- board text added: "HardDuino"
- board text removed: "Harduino"
