File: template/Harduino.kicad_pcb (KiCad board)
At the start: 2 copper layers, 40.6 x 40.6 mm, 24 parts, among them J1 2, J10 11, J11 12, J12 13, J13 A0, J14 A1, J15 A2, J16 A3, J17 A4, J18 A5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

Commit message: Add description Fix template
Other:
- board text added: "10"
- board text added: "11"
- board text added: "12"
- board text added: "13"
- board text added: "2"
- board text added: "3"
- board text added: "4"
- board text added: "5"
- board text added: "6"
- board text added: "7"
- board text added: "8"
- board text added: "9"
- board text added: "A0"
- board text added: "A1"
- board text added: "A2"
- board text added: "A3"
- board text added: "A4"
- board text added: "A5"
- board text added: "Gnd"
- board text added: "Harduino"
- board text added: "Vcc"
Changed lines of the file:
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@@
   (general
     (thickness 1.6)
-    (drawings 8)
+    (drawings 29)
     (tracks 0)
     (zones 0)
@@
     )
   )
+  (gr_text Harduino (at 109.22 52.07) (layer F.SilkS)
+    (effects (font (size 1 1) (thickness 0.15)))
+  )
+  (gr_text Gnd (at 90.17 82.55) (layer F.SilkS)
+    (effects (font (size 1 1) (thickness 0.15)))
+  )
+  (gr_text A5 (at 90.17 80.01) (layer F.SilkS)
+    (effects (font (size 1 1) (thickness 0.15)))
+  )
+  (gr_text A4 (at 90.17 77.47) (layer F.SilkS)
+    (effects (font (size 1 1) (thickness 0.15)))
+  )
+  (gr_text A3 (at 90.17 74.93) (layer F.SilkS)
+    (effects (font (size 1 1) (thickness 0.15)))
+  )
+  (gr_text A2 (at 90.17 72.39) (layer F.SilkS)
+    (effects (font (size 1 1) (thickness 0.15)))
+  )
+  (gr_text A1 (at 90.17 69.85) (layer F.SilkS)
+    (effects (font (size 1 1) (thickness 0.15)))
+  )
+  (gr_text A0 (at 90.17 67.31) (layer F.SilkS)
+    (effects (font (size 1 1) (thickness 0.15)))
+  )
+  (gr_text Vcc (at 90.17 59.69) (layer F.SilkS)
+    (effects (font (size 1 1) (thickness 0.15)))
+  )
+  (gr_text 13 (at 90.17 64.77) (layer F.SilkS)
+    (effects (font (size 1 1) (thickness 0.15)))
+  )
+  (gr_text 12 (at 90.17 62.23) (layer F.SilkS)
+    (effects (font (size 1 1) (thickness 0.15)))
+  )
+  (gr_text 11 (at 128.27 59.69) (layer F.SilkS)
+    (effects (font (size 1 1) (thickness 0.15)))
+  )
+  (gr_text 10 (at 128.27 62.23) (layer F.SilkS)
+    (effects (font (size 1 1) (thickness 0.15)))
+  )
+  (gr_text 9 (at 128.27 64.77) (layer F.SilkS)
+    (effects (font (size 1 1) (thickness 0.15)))
+  )
+  (gr_text 8 (at 128.27 67.31) (layer F.SilkS)
+    (effects (font (size 1 1) (thickness 0.15)))
+  )
+  (gr_text 7 (at 128.27 69.85) (layer F.SilkS)
+    (effects (font (size 1 1) (thickness 0.15)))
+  )
+  (gr_text 6 (at 128.27 72.39) (layer F.SilkS)
+    (effects (font (size 1 1) (thickness 0.15)))
+  )
+  (gr_text 5 (at 128.27 74.93) (layer F.SilkS)
+    (effects (font (size 1 1) (thickness 0.15)))
+  )
+  (gr_text 4 (at 128.27 77.47) (layer F.SilkS)
+    (effects (font (size 1 1) (thickness 0.15)))
+  )
+  (gr_text 3 (at 128.27 80.01) (layer F.SilkS)
+    (effects (font (size 1 1) (thickness 0.15)))
+  )
+  (gr_text 2 (at 128.27 82.55) (layer F.SilkS)
+    (effects (font (size 1 1) (thickness 0.15)))
+  )
   (gr_arc (start 127 53.34) (end 129.54 53.34) (angle -90) (layer Edge.Cuts) (width 0.15))

Commit message: Harduino -> HardDuino
Other:
- board text added: "HardDuino"
- board text removed: "Harduino"
Changed lines of the file:
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@@
     )
   )
-  (gr_text Harduino (at 109.22 52.07) (layer F.SilkS)
+  (gr_text HardDuino (at 109.22 52.07) (layer F.SilkS)
     (effects (font (size 1 1) (thickness 0.15)))
   )
