File: modules/Pins/Pins.kicad_pcb (KiCad board)
At the start: 2 copper layers, 40.6 x 40.6 mm, 25 parts, among them J1 2, J10 11, J11 12, J12 13, J13 A0, J14 A1, J15 A2, J16 A3, J17 A4, J18 A5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

Commit message: Add some pinheaders
Parts:
- added J22: Conn_01x10_Male, Connector_PinHeader_2.54mm:PinHeader_1x10_P2.54mm_Vertical, F.Cu at (115.6, 80.0)
- added J23: Conn_01x10_Male, Connector_PinHeader_2.54mm:PinHeader_1x10_P2.54mm_Vertical, F.Cu at (118.1, 80.0)
- added J24: Conn_01x06_Male, Connector_PinHeader_2.54mm:PinHeader_1x06_P2.54mm_Vertical, F.Cu at (102.9, 67.3)
- added J25: Conn_01x06_Male, Connector_PinHeader_2.54mm:PinHeader_1x06_P2.54mm_Vertical, F.Cu at (100.3, 67.3)
- added J26: Conn_01x06_Male, Connector_PinHeader_2.54mm:PinHeader_1x06_P2.54mm_Vertical, F.Cu at (97.8, 67.3)
- moved J21 26.2 mm to (120.7, 80.0), turned to 180 degrees
Connections:
- J21 pad 10: Net-(J21-Pad10) -> Net-(J12-Pad1)
- J21 pad 8: Net-(J21-Pad8) -> Net-(J10-Pad1)
- J21 pad 9: Net-(J21-Pad9) -> Net-(J11-Pad1)
- J3 pad 1: Net-(J3-Pad1) -> Net-(J21-Pad1)
- J4 pad 1: Net-(J4-Pad1) -> Net-(J21-Pad2)
- J5 pad 1: Net-(J5-Pad1) -> Net-(J21-Pad3)
- J6 pad 1: Net-(J6-Pad1) -> Net-(J21-Pad4)
- J7 pad 1: Net-(J7-Pad1) -> Net-(J21-Pad5)
- J8 pad 1: Net-(J8-Pad1) -> Net-(J21-Pad6)
- J9 pad 1: Net-(J9-Pad1) -> Net-(J21-Pad7)

Commit message: Pins (sensor) shield ready
Parts:
- added J27: Conn_01x04_Male, Connector_PinHeader_2.54mm:PinHeader_1x04_P2.54mm_Vertical, F.Cu at (99.1, 61.0)
- added J28: Conn_01x04_Male, Connector_PinHeader_2.54mm:PinHeader_1x04_P2.54mm_Vertical, F.Cu at (104.1, 61.0)
- added J29: Conn_01x04_Male, Connector_PinHeader_2.54mm:PinHeader_1x04_P2.54mm_Vertical, F.Cu at (109.2, 61.0)
- added J30: Conn_01x06_Male, Connector_PinHeader_2.54mm:PinHeader_1x06_P2.54mm_Vertical, F.Cu at (109.2, 85.1)
- added J31: Conn_01x06_Male, Connector_PinHeader_2.54mm:PinHeader_1x06_P2.54mm_Vertical, F.Cu at (106.7, 85.1)
- added JP1: Jumper_3_Bridged12, Connector_PinHeader_2.54mm:PinHeader_1x03_P2.54mm_Vertical, F.Cu at (120.7, 87.6)
- added RN1: R_Network06, Resistor_THT:R_Array_SIP7, F.Cu at (111.8, 87.6)
- J21, J22, J23: value Conn_01x10_Male -> Conn_01x12_Male; footprint Connector_PinHeader_2.54mm:PinHeader_1x10_P2.54mm_Vertical -> Connector_PinHeader_2.54mm:PinHeader_1x12_P2.54mm_Vertical
- moved J22 3.59 mm to (118.1, 82.5)
- moved J23 3.59 mm to (115.6, 82.5)
- moved J21 2.54 mm to (120.7, 82.5)
Connections:
- net Net-(J17-Pad1) renamed /SDA
- net Net-(J18-Pad1) renamed /SCL
- J21 pad 1: Net-(J21-Pad1) -> Net-(J1-Pad1)
- J21 pad 10: Net-(J12-Pad1) -> Net-(J10-Pad1)
- J21 pad 2: Net-(J21-Pad2) -> Net-(J2-Pad1)
- J21 pad 8: Net-(J10-Pad1) -> Net-(J21-Pad8)
- J21 pad 9: Net-(J11-Pad1) -> Net-(J21-Pad9)
- J22 pad 1: GND -> VCC
- J22 pad 10: GND -> VCC
- J22 pad 2: GND -> VCC
- J22 pad 3: GND -> VCC
- J22 pad 4: GND -> VCC
- J22 pad 5: GND -> VCC
- J22 pad 6: GND -> VCC
- J22 pad 7: GND -> VCC
- J22 pad 8: GND -> VCC
- J22 pad 9: GND -> VCC
- J23 pad 1: VCC -> GND
- J23 pad 10: VCC -> GND
- J23 pad 2: VCC -> GND
- J23 pad 3: VCC -> GND
- J23 pad 4: VCC -> GND
- J23 pad 5: VCC -> GND
- J23 pad 6: VCC -> GND
- J23 pad 7: VCC -> GND
- J23 pad 8: VCC -> GND
- J23 pad 9: VCC -> GND
- J3 pad 1: Net-(J21-Pad1) -> Net-(J21-Pad3)
- J4 pad 1: Net-(J21-Pad2) -> Net-(J21-Pad4)
- J5 pad 1: Net-(J21-Pad3) -> Net-(J21-Pad5)
- J6 pad 1: Net-(J21-Pad4) -> Net-(J21-Pad6)
- J7 pad 1: Net-(J21-Pad5) -> Net-(J21-Pad7)
- J8 pad 1: Net-(J21-Pad6) -> Net-(J21-Pad8)
- J9 pad 1: Net-(J21-Pad7) -> Net-(J21-Pad9)
Routing:
- net GND: track 0.00 -> 113.2 mm
- net VCC: track 0.00 -> 95.9 mm
- net Net-(J12-Pad1): track 0.00 -> 48.4 mm, vias 0 -> 1
- net /SDA: track 0.00 -> 42.4 mm
- net /SCL: track 0.00 -> 40.2 mm
- net Net-(J11-Pad1): track 0.00 -> 39.3 mm, vias 0 -> 1
- net Net-(JP1-Pad2): track 0.00 -> 10.0 mm
- net Net-(J16-Pad1): track 0.00 -> 5.08 mm
- net Net-(J15-Pad1): track 0.00 -> 5.08 mm
- net Net-(J14-Pad1): track 0.00 -> 5.08 mm
- net Net-(J13-Pad1): track 0.00 -> 5.08 mm
- net Net-(J30-Pad6): track 0.00 -> 5.08 mm
- net Net-(J30-Pad5): track 0.00 -> 5.08 mm
- net Net-(J30-Pad4): track 0.00 -> 5.08 mm
- net Net-(J30-Pad3): track 0.00 -> 5.08 mm
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Other:
- board text added: "A0-A5"
- board text added: "D2-D13"
- board text added: "I2C"
- board text added: "PullUps"
- board text added: "SCL"
- board text added: "SDA"
