File: modules/h2xS/h2xS.sch (KiCad schematic (older format))
At the start: 51 parts, among them J1 2, J10 11, J1001 Conn_01x04_Male, J1002 Conn_01x12_Male, J1003 Conn_01x04_Male, J1004 Conn_01x12_Male, J1005 Conn_01x12_Male, J1006 Conn_01x06_Male, J1007 Barrel_Jack_MountingPin, J11 12, J12 13, J13 A0, J14 A1, J15 A2, J16 A3, J17 A4, J18 A5, J19 Vcc, J2 3, J20 Gnd, J3 4, J4 5, J5 6, J6 7, J7 8, J8 9, J9 10

Commit message: h2x with Sensor Shield in work
Parts:
- removed J1001, J1003: Conn_01x04_Male, Connector_PinHeader_2.54mm:PinHeader_1x04_P2.54mm_Vertical, symbol Connector:Conn_01x04_Male
- removed J1002, J1004, J1005: Conn_01x12_Male, Connector_PinHeader_2.54mm:PinHeader_1x12_P2.54mm_Vertical, symbol Connector:Conn_01x12_Male
- removed J1006: Conn_01x06_Male, Connector_PinHeader_2.54mm:PinHeader_1x06_P2.54mm_Vertical, symbol Connector:Conn_01x06_Male
- removed J1007: Barrel_Jack_MountingPin, Connector_BarrelJack:BarrelJack_Horizontal, symbol Connector:Barrel_Jack_MountingPin
- removed JO1: 2, Connector_PinHeader_2.54mm:PinHeader_1x01_P2.54mm_Vertical, symbol Connector:Conn_01x01_Male
- removed JO10: 11, Connector_PinHeader_2.54mm:PinHeader_1x01_P2.54mm_Vertical, symbol Connector:Conn_01x01_Male
- removed JO11: 12, Connector_PinHeader_2.54mm:PinHeader_1x01_P2.54mm_Vertical, symbol Connector:Conn_01x01_Male
- removed JO12: 13, Connector_PinHeader_2.54mm:PinHeader_1x01_P2.54mm_Vertical, symbol Connector:Conn_01x01_Male
- removed JO13: A0, Connector_PinHeader_2.54mm:PinHeader_1x01_P2.54mm_Vertical, symbol Connector:Conn_01x01_Male
- removed JO14: A1, Connector_PinHeader_2.54mm:PinHeader_1x01_P2.54mm_Vertical, symbol Connector:Conn_01x01_Male
- removed JO15: A2, Connector_PinHeader_2.54mm:PinHeader_1x01_P2.54mm_Vertical, symbol Connector:Conn_01x01_Male
- removed JO16: A3, Connector_PinHeader_2.54mm:PinHeader_1x01_P2.54mm_Vertical, symbol Connector:Conn_01x01_Male
- removed JO17: A4, Connector_PinHeader_2.54mm:PinHeader_1x01_P2.54mm_Vertical, symbol Connector:Conn_01x01_Male
- removed JO18: A5, Connector_PinHeader_2.54mm:PinHeader_1x01_P2.54mm_Vertical, symbol Connector:Conn_01x01_Male
- removed JO19: Vcc, Connector_PinHeader_2.54mm:PinHeader_1x01_P2.54mm_Vertical, symbol Connector:Conn_01x01_Male
- removed JO2: 3, Connector_PinHeader_2.54mm:PinHeader_1x01_P2.54mm_Vertical, symbol Connector:Conn_01x01_Male
- removed JO20: Gnd, Connector_PinHeader_2.54mm:PinHeader_1x01_P2.54mm_Vertical, symbol Connector:Conn_01x01_Male
- removed JO3: 4, Connector_PinHeader_2.54mm:PinHeader_1x01_P2.54mm_Vertical, symbol Connector:Conn_01x01_Male
- removed JO4: 5, Connector_PinHeader_2.54mm:PinHeader_1x01_P2.54mm_Vertical, symbol Connector:Conn_01x01_Male
- removed JO5: 6, Connector_PinHeader_2.54mm:PinHeader_1x01_P2.54mm_Vertical, symbol Connector:Conn_01x01_Male
- removed JO6: 7, Connector_PinHeader_2.54mm:PinHeader_1x01_P2.54mm_Vertical, symbol Connector:Conn_01x01_Male
- removed JO7: 8, Connector_PinHeader_2.54mm:PinHeader_1x01_P2.54mm_Vertical, symbol Connector:Conn_01x01_Male
- removed JO8: 9, Connector_PinHeader_2.54mm:PinHeader_1x01_P2.54mm_Vertical, symbol Connector:Conn_01x01_Male
- removed JO9: 10, Connector_PinHeader_2.54mm:PinHeader_1x01_P2.54mm_Vertical, symbol Connector:Conn_01x01_Male
- added H5, H6, H7, H8: MountingHole, MountingHole:MountingHole_3.2mm_M3, symbol Mechanical:MountingHole
- added J21, J27: Conn_01x10_Male, Connector_PinSocket_2.54mm:PinSocket_1x10_P2.54mm_Vertical, symbol Connector:Conn_01x10_Male
- added J22, J23, J26: Conn_01x12_Male, Connector_PinHeader_2.54mm:PinHeader_1x12_P2.54mm_Vertical, symbol Connector:Conn_01x12_Male
- added J24, J25: Conn_01x04_Male, Connector_PinHeader_2.54mm:PinHeader_1x04_P2.54mm_Vertical, symbol Connector:Conn_01x04_Male
- added J28: Conn_01x06_Male, Connector_PinHeader_2.54mm:PinHeader_1x06_P2.54mm_Vertical, symbol Connector:Conn_01x06_Male
- added J29: Barrel_Jack_Switch, Connector_BarrelJack:BarrelJack_Horizontal, symbol Connector:Barrel_Jack_Switch
Connections:
- net at J1.1 (Pin_1): now also J21.1 (Pin_1), J22.1 (Pin_1)
- net at J2.1 (Pin_1): now also J21.2 (Pin_2), J22.2 (Pin_2)
- net at J3.1 (Pin_1): now also J21.3 (Pin_3), J22.3 (Pin_3)
- net at J4.1 (Pin_1): now also J21.4 (Pin_4), J22.4 (Pin_4)
- net at J5.1 (Pin_1): now also J21.5 (Pin_5), J22.5 (Pin_5)
- net at J6.1 (Pin_1): now also J21.6 (Pin_6), J22.6 (Pin_6)
- net at J7.1 (Pin_1): now also J21.7 (Pin_7), J22.7 (Pin_7)
- net at J8.1 (Pin_1): now also J21.8 (Pin_8), J22.8 (Pin_8)
- net at J9.1 (Pin_1): now also J21.9 (Pin_9), J22.9 (Pin_9)
- net at J10.1 (Pin_1): now also J21.10 (Pin_10), J22.10 (Pin_10)
- net at J11.1 (Pin_1): now also J22.11 (Pin_11), J27.2 (Pin_2)
- net at J13.1 (Pin_1): now also J27.4 (Pin_4), J28.1 (Pin_1)
- net at J14.1 (Pin_1): now also J27.5 (Pin_5), J28.2 (Pin_2)
- net at J15.1 (Pin_1): now also J27.6 (Pin_6), J28.3 (Pin_3)
- net at J16.1 (Pin_1): now also J27.7 (Pin_7), J28.4 (Pin_4)
- net at J17.1 (Pin_1): now also J24.2 (Pin_2), J25.2 (Pin_2), J27.8 (Pin_8), J28.5 (Pin_5)
- net at J18.1 (Pin_1): now also J24.1 (Pin_1), J25.1 (Pin_1), J27.9 (Pin_9), J28.6 (Pin_6)
- net VCC: now reaches J19.1 (Pin_1)
- net VCC: now also J23.1 (Pin_1), J23.10 (Pin_10), J23.11 (Pin_11), J23.12 (Pin_12), J23.2 (Pin_2), J23.3 (Pin_3), J23.4 (Pin_4), J23.5 (Pin_5), J23.6 (Pin_6), J23.7 (Pin_7), J23.8 (Pin_8), J23.9 (Pin_9), J24.3 (Pin_3), J25.3 (Pin_3), J27.1 (Pin_1), J29.1
- net GND: now reaches J20.1 (Pin_1)
- net GND: now also J24.4 (Pin_4), J25.4 (Pin_4), J26.1 (Pin_1), J26.10 (Pin_10), J26.11 (Pin_11), J26.12 (Pin_12), J26.2 (Pin_2), J26.3 (Pin_3), J26.4 (Pin_4), J26.5 (Pin_5), J26.6 (Pin_6), J26.7 (Pin_7), J26.8 (Pin_8), J26.9 (Pin_9), J27.10 (Pin_10), J29.2
- net at J12.1 (Pin_1): now also J22.12 (Pin_12), J27.3 (Pin_3)
Other:
- note added: "Gnd"
- note added: "SCL"
- note added: "SDA"
- note added: "Vcc"

Commit message: Sensor Shield ready
Connections:
- net 2: now reaches J1.1 (Pin_1), J21.1 (Pin_1), J22.1 (Pin_1)
- net 3: now reaches J2.1 (Pin_1), J21.2 (Pin_2), J22.2 (Pin_2)
- net 4: now reaches J21.3 (Pin_3), J22.3 (Pin_3), J3.1 (Pin_1)
- net 5: now reaches J21.4 (Pin_4), J22.4 (Pin_4), J4.1 (Pin_1)
- net 6: now reaches J21.5 (Pin_5), J22.5 (Pin_5), J5.1 (Pin_1)
- net 7: now reaches J21.6 (Pin_6), J22.6 (Pin_6), J6.1 (Pin_1)
- net 8: now reaches J21.7 (Pin_7), J22.7 (Pin_7), J7.1 (Pin_1)
- net 9: now reaches J21.8 (Pin_8), J22.8 (Pin_8), J8.1 (Pin_1)
- net 10: now reaches J21.9 (Pin_9), J22.9 (Pin_9), J9.1 (Pin_1)
- net 11: now reaches J10.1 (Pin_1), J21.10 (Pin_10), J22.10 (Pin_10)
- net 12: now reaches J11.1 (Pin_1), J22.11 (Pin_11), J27.2 (Pin_2)
- net A0: now reaches J13.1 (Pin_1), J27.4 (Pin_4), J28.1 (Pin_1)
- net A1: now reaches J14.1 (Pin_1), J27.5 (Pin_5), J28.2 (Pin_2)
- net A2: now reaches J15.1 (Pin_1), J27.6 (Pin_6), J28.3 (Pin_3)
- net A3: now reaches J16.1 (Pin_1), J27.7 (Pin_7), J28.4 (Pin_4)
- net A4: now reaches J17.1 (Pin_1), J24.2 (Pin_2), J25.2 (Pin_2), J27.8 (Pin_8), J28.5 (Pin_5)
- net A5: now reaches J18.1 (Pin_1), J24.1 (Pin_1), J25.1 (Pin_1), J27.9 (Pin_9), J28.6 (Pin_6)
- net 13: now reaches J12.1 (Pin_1), J22.12 (Pin_12), J27.3 (Pin_3)
Changed lines of the file:
@@
 Wire Wire Line
 	3050 4825 3050 4925
+Text Label 1375 2500 0    50   ~ 0
+2
+Text Label 1375 2600 0    50   ~ 0
+3
+Text Label 1375 2700 0    50   ~ 0
+4
+Text Label 1400 2800 0    50   ~ 0
+5
+Text Label 1425 2900 0    50   ~ 0
+6
+Text Label 1425 3000 0    50   ~ 0
+7
+Text Label 1450 3100 0    50   ~ 0
+8
+Text Label 1475 3200 0    50   ~ 0
+9
+Text Label 1500 3300 0    50   ~ 0
+10
+Text Label 1525 3400 0    50   ~ 0
+11
+Text Label 1525 4000 0    50   ~ 0
+12
+Text Label 1525 4150 0    50   ~ 0
+13
+Text Label 6225 2500 0    50   ~ 0
+A0
+Text Label 6225 2600 0    50   ~ 0
+A1
+Text Label 6225 2700 0    50   ~ 0
+A2
+Text Label 6225 2800 0    50   ~ 0
+A3
+Text Label 6225 2900 0    50   ~ 0
+A4
+Text Label 6225 3000 0    50   ~ 0
+A5
 $EndSCHEMATC
