File: modules/h2xSv2/h2xSv2.kicad_pcb (KiCad board)
At the start: 2 copper layers, 95.2 x 40.6 mm, 18 parts, among them J1 Conn_01x10_Male, J10 Conn_01x02_Male, J2 Conn_01x10_Male, J3 Conn_01x10_Male, J4 Conn_01x10_Male, J5 Conn_01x04_Male, J6 Conn_01x04_Male, J7 Conn_01x12_Male, J8 Conn_01x12_Male, J9 Conn_01x12_Male

Commit message: Silk
Other:
- board text added: "I2C"
- board text added: "SCL"
- board text added: "SDA"
Changed lines of the file:
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@@
   (general
     (thickness 1.6)
-    (drawings 32)
+    (drawings 62)
     (tracks 4)
     (zones 0)
@@
     (tags "mounting hole 3.2mm no annular m3")
     (attr virtual)
-    (fp_text reference H1 (at -3.81 -4.2) (layer F.SilkS) hide
+    (fp_text reference H1 (at 5.08 -2.54) (layer F.SilkS) hide
       (effects (font (size 1 1) (thickness 0.15)))
     )
@@
     (tags "mounting hole 3.2mm no annular m3")
     (attr virtual)
-    (fp_text reference H2 (at -3.81 3.81) (layer F.SilkS) hide
+    (fp_text reference H2 (at -3.175 3.81) (layer F.SilkS) hide
       (effects (font (size 1 1) (thickness 0.15)))
     )
@@
     (tags "mounting hole 3.2mm no annular m3")
     (attr virtual)
-    (fp_text reference H3 (at 3.81 -3.81) (layer F.SilkS) hide
+    (fp_text reference H3 (at -3.175 3.81) (layer F.SilkS) hide
       (effects (font (size 1 1) (thickness 0.15)))
     )
@@
     (tags "mounting hole 3.2mm no annular m3")
     (attr virtual)
-    (fp_text reference H4 (at 3.81 3.81) (layer F.SilkS) hide
+    (fp_text reference H4 (at 3.175 3.81) (layer F.SilkS) hide
       (effects (font (size 1 1) (thickness 0.15)))
     )
@@
     (tags "mounting hole 3.2mm no annular m3")
     (attr virtual)
-    (fp_text reference H5 (at 0 -4.2) (layer F.SilkS)
+    (fp_text reference H5 (at -3.81 -3.175) (layer F.SilkS) hide
       (effects (font (size 1 1) (thickness 0.15)))
     )
@@
     (tags "mounting hole 3.2mm no annular m3")
     (attr virtual)
-    (fp_text reference H6 (at 0 -4.2) (layer F.SilkS)
+    (fp_text reference H6 (at -3.81 -3.175) (layer F.SilkS) hide
       (effects (font (size 1 1) (thickness 0.15)))
     )
@@
     (tags "mounting hole 3.2mm no annular m3")
     (attr virtual)
-    (fp_text reference H7 (at 0 -4.2) (layer F.SilkS)
+    (fp_text reference H7 (at 4.445 2.54) (layer F.SilkS) hide
       (effects (font (size 1 1) (thickness 0.15)))
     )
@@
     (tags "mounting hole 3.2mm no annular m3")
     (attr virtual)
-    (fp_text reference H8 (at 0 -4.2) (layer F.SilkS)
+    (fp_text reference H8 (at -3.81 3.175) (layer F.SilkS) hide
       (effects (font (size 1 1) (thickness 0.15)))
     )
@@
     (pad 1 np_thru_hole circle (at 0 0) (size 3.2 3.2) (drill 3.2) (layers *.Cu *.Mask))
   )
+  (gr_text 2 (at 115.57 90.17 270) (layer F.SilkS)
+    (effects (font (size 1 1) (thickness 0.15)))
+  )
+  (gr_text 3 (at 118.11 90.17 270) (layer F.SilkS)
+    (effects (font (size 1 1) (thickness 0.15)))
+  )
+  (gr_text 4 (at 120.65 90.17 270) (layer F.SilkS)
+    (effects (font (size 1 1) (thickness 0.15)))
+  )
+  (gr_text 5 (at 123.19 90.17 270) (layer F.SilkS)
+    (effects (font (size 1 1) (thickness 0.15)))
+  )
+  (gr_text 6 (at 125.73 90.17 270) (layer F.SilkS)
+    (effects (font (size 1 1) (thickness 0.15)))
+  )
+  (gr_text 7 (at 128.27 90.17 270) (layer F.SilkS)
+    (effects (font (size 1 1) (thickness 0.15)))
+  )
+  (gr_text 8 (at 130.81 90.17 270) (layer F.SilkS)
+    (effects (font (size 1 1) (thickness 0.15)))
+  )
+  (gr_text 9 (at 133.35 90.17 270) (layer F.SilkS)
+    (effects (font (size 1 1) (thickness 0.15)))
+  )
+  (gr_text 10 (at 135.89 90.17 270) (layer F.SilkS)
+    (effects (font (size 1 1) (thickness 0.15)))
+  )
+  (gr_text 11 (at 138.43 90.17 270) (layer F.SilkS)
+    (effects (font (size 1 1) (thickness 0.15)))
+  )
+  (gr_text 12 (at 135.89 52.07 270) (layer F.SilkS)
+    (effects (font (size 1 1) (thickness 0.15)))
+  )
+  (gr_text 13 (at 133.35 52.07 270) (layer F.SilkS)
+    (effects (font (size 1 1) (thickness 0.15)))
+  )
+  (gr_text Vcc (at 139.065 46.99 270) (layer F.SilkS)
+    (effects (font (size 1 1) (thickness 0.15)))
+  )
+  (gr_text A0 (at 130.81 52.07 270) (layer F.SilkS)
+    (effects (font (size 1 1) (thickness 0.15)))
+  )
+  (gr_text A1 (at 128.27 52.07 270) (layer F.SilkS)
+    (effects (font (size 1 1) (thickness 0.15)))
+  )
+  (gr_text A2 (at 125.73 52.07 270) (layer F.SilkS)
+    (effects (font (size 1 1) (thickness 0.15)))
+  )
+  (gr_text A3 (at 123.19 52.07 270) (layer F.SilkS)
+    (effects (font (size 1 1) (thickness 0.15)))
+  )
+  (gr_text A4 (at 120.65 52.07 270) (layer F.SilkS)
+    (effects (font (size 1 1) (thickness 0.15)))
+  )
+  (gr_text A5 (at 118.11 52.07 270) (layer F.SilkS)
+    (effects (font (size 1 1) (thickness 0.15)))
+  )
+  (gr_text Gnd (at 115.57 52.07 270) (layer F.SilkS)
+    (effects (font (size 1 1) (thickness 0.15)))
+  )
+  (gr_line (start 146.05 62.865) (end 148.59 57.21) (layer F.SilkS) (width 0.12))
   (gr_poly (pts (xy 102.32 67.435) (xy 103.03 68.455) (xy 103.25 68.775) (xy 103.44 68.955) (xy 103.5 68.995) (xy 103.93 69.125) (xy 103.97 69.105) (xy 103.97 69.015) (xy 103.78 68.585) (xy 103.48 67.935) (xy 104.29 68.925) (xy 104.49 69.145) (xy 104.61 69.245) (xy 104.69 69.275) (xy 104.87 69.285) (xy 105.09 69.345) (xy 105.05 69.225) (xy 104.54 68.335) (xy 105.31 69.175) (xy 105.47 69.365) (xy 105.56 69.445) (xy 105.67 69.495) (xy 106.11 69.545) (xy 106.57 69.565) (xy 107.05 68.965) (xy 107.2 68.815) (xy 107.19 68.895) (xy 107.05 69.225) (xy 106.97 69.395) (xy 106.96 69.475) (xy 107.04 69.485) (xy 107.44 69.465) (xy 107.79 69.355) (xy 108.46 68.785) (xy 108.34 69.075) (xy 107.91 69.725) (xy 107.58 69.785) (xy 106.97 69.835) (xy 106.78 69.905) (xy 107 69.965) (xy 108.33 70.185) (xy 108.65 70.255) (xy 108.78 70.355) (xy 108.8 70.525) (xy 108.78 70.685) (xy 108.72 70.765) (xy 108.67 70.785) (xy 108.63 70.865) (xy 108.63 70.965) (xy 108.57 71.015) (xy 108.38 71.065) (xy 107.76 71.175) (xy 107.47 71.255) (xy 107.34 71.375) (xy 107.31 71.435) (xy 107.28 71.585) (xy 107.29 71.755) (xy 106.96 75.525) (xy 107.01 72.135) (xy 107 71.855) (xy 106.99 71.665) (xy 106.98 71.625) (xy 106.94 71.585) (xy 106.89 71.705) (xy 106.86 72.035) (xy 106.83 72.525) (xy 106.8 73.905) (xy 106.78 74.435) (xy 106.74 74.765) (xy 106.71 74.585) (xy 106.68 73.905) (xy 106.68 73.025) (xy 106.66 71.805) (xy 106.5 71.845) (xy 106.39 71.845) (xy 106.32 71.795) (xy 106.25 71.665) (xy 106.01 71.035) (xy 106.32 70.635) (xy 106.28 70.865) (xy 106.27 71.025) (xy 106.27 71.095) (xy 106.34 71.225) (xy 106.49 71.435) (xy 107.4 71.045) (xy 107.53 70.975) (xy 107.58 70.915) (xy 107.47 70.875) (xy 107.68 70.835) (xy 108.2 70.825) (xy 108.32 70.805) (xy 108.41 70.755) (xy 108.44 70.695) (xy 108.41 70.575) (xy 108.25 70.475) (xy 107.98 70.365) (xy 107.58 70.285) (xy 107.34 70.275) (xy 107.2 70.295) (xy 107.15 70.335) (xy 107.08 70.435) (xy 107.03 70.445) (xy 106.97 70.445) (xy 106.85 70.395) (xy 106.7 70.295) (xy 106.66 70.235) (xy 106.65 70.195) (xy 106.59 70.165) (xy 106.51 70.135) (xy 106.02 70.115) (xy 105.57 70.125) (xy 105.43 70.145) (xy 105.31 70.175) (xy 105.33 70.215) (xy 105.54 70.255) (xy 105.84 70.275) (xy 106.35 70.285) (xy 105.93 70.435) (xy 105.93 70.465) (xy 106.13 70.485) (xy 106.14 70.515) (xy 105.9 70.635) (xy 105.84 70.705) (xy 105.71 70.895) (xy 105.51 71.325) (xy 105.08 72.375) (xy 104.86 73.025) (xy 104.81 73.195) (xy 104.78 73.335) (xy 104.83 73.415) (xy 104.88 73.385) (xy 104.92 73.315) (xy 105.01 73.095) (xy 105.19 72.585) (xy 105.5 71.755) (xy 105.46 72.015) (xy 105.21 73.015) (xy 105.15 73.225) (xy 105.09 73.565) (xy 105.07 73.685) (xy 105.07 73.795) (xy 105.12 73.855) (xy 105.18 73.775) (xy 105.22 73.625) (xy 105.32 73.255) (xy 105.48 72.535) (xy 105.51 72.535) (xy 105.36 73.695) (xy 105.29 74.145) (xy 105.68 74.715) (xy 105.84 75.015) (xy 105.23 74.305) (xy 104.53 73.415) (xy 102.89 73.485) (xy 104.29 73.185) (xy 104.5 73.115) (xy 104.58 72.895) (xy 104.87 72.015) (xy 105.12 71.165) (xy 105.28 70.495) (xy 104.55 69.925) (xy 104.91 69.885) (xy 105.36 69.905) (xy 105.84 69.915) (xy 103.92 69.495) (xy 103.12 69.305) (xy 102.69 68.335)) (layer F.SilkS) (width 0.1))
-  (gr_text HardDuino (at 109.22 52.07) (layer F.SilkS)
+  (gr_text HardDuino (at 105.41 61.595) (layer F.SilkS)
     (effects (font (size 1 1) (thickness 0.15)))
   )
@@
     (effects (font (size 1 1) (thickness 0.15)))
   )
+  (gr_text I2C (at 141.605 61.595) (layer F.SilkS)
+    (effects (font (size 1 1) (thickness 0.15)))
+  )
+  (gr_line (start 137.795 66.675) (end 137.795 62.865) (layer F.SilkS) (width 0.12))
+  (gr_line (start 146.05 66.675) (end 137.795 66.675) (layer F.SilkS) (width 0.12))
+  (gr_line (start 146.05 62.865) (end 146.05 66.675) (layer F.SilkS) (width 0.12))
+  (gr_line (start 137.795 62.865) (end 146.05 62.865) (layer F.SilkS) (width 0.12))
+  (gr_text Gnd (at 144.78 64.77 90) (layer F.SilkS)
+    (effects (font (size 1 1) (thickness 0.15)))
+  )
+  (gr_text Vcc (at 142.875 64.77 90) (layer F.SilkS)
+    (effects (font (size 1 1) (thickness 0.15)))
+  )
+  (gr_text SCL (at 139.065 64.77 90) (layer F.SilkS)
+    (effects (font (size 1 1) (thickness 0.15)))
+  )
+  (gr_text SDA (at 140.97 64.77 90) (layer F.SilkS)
+    (effects (font (size 1 1) (thickness 0.15)))
+  )

Commit message: Copy&paste some tracks from old pcb
Parts:
- moved J10 30.9 mm to (57.1, 34.9)
- moved J7 30.9 mm to (141.0, 59.7)
- moved J8 30.9 mm to (143.5, 59.7)
- moved J9 30.9 mm to (146.1, 59.7)
- moved H3 30.9 mm to (57.1, 25.4)
- moved H4 30.9 mm to (90.2, 25.4)
- moved H5 30.9 mm to (133.3, 25.4)
- moved H6 30.9 mm to (100.3, 25.4)
- moved J1 30.9 mm to (85.1, 25.4)
- moved J3 30.9 mm to (128.3, 25.4)
- moved J5 30.9 mm to (138.4, 26.7)
- moved J6 30.9 mm to (138.4, 23.5)
- moved H1 30.9 mm to (57.1, 58.4)
- moved H2 30.9 mm to (90.2, 58.4)
- moved H7 30.9 mm to (133.3, 58.4)
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Routing:
- net /A5: track 0.00 -> 71.3 mm, vias 0 -> 1
- net /A4: track 0.00 -> 69.4 mm, vias 0 -> 1
- net /2: track 0.00 -> 68.6 mm, vias 0 -> 1
- net /3: track 0.00 -> 66.7 mm, vias 0 -> 1
- net /A3: track 0.00 -> 65.9 mm, vias 0 -> 1
- net /4: track 0.00 -> 64.8 mm, vias 0 -> 1
- net /5: track 0.00 -> 62.9 mm, vias 0 -> 1
- net /A1: track 0.00 -> 61.9 mm, vias 0 -> 1
- net /A2: track 2.54 -> 64.0 mm, vias 0 -> 1
- net /13: track 0.00 -> 61.1 mm, vias 0 -> 2
- net /6: track 0.00 -> 61.0 mm, vias 0 -> 1
- net /12: track 0.00 -> 60.6 mm, vias 0 -> 2
- net /A0: track 0.00 -> 60.2 mm, vias 0 -> 1
- net /7: track 0.00 -> 59.1 mm, vias 0 -> 1
- net /8: track 0.00 -> 57.2 mm, vias 0 -> 1
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
Commit message: h2xS v2 in work
Parts:
- added J11: Conn_01x06_Male, Connector_PinHeader_2.54mm:PinHeader_1x06_P2.54mm_Vertical, F.Cu at (64.8, 22.9)
Routing:
- net VCC: track 0.00 -> 136.5 mm, vias 0 -> 1
- net /2: track 68.6 -> 107.7 mm
- net GND: track 11.3 -> 47.5 mm
- net /3: track 66.7 -> 102.6 mm
- net /4: track 64.8 -> 97.5 mm
- net /5: track 62.9 -> 92.8 mm
- net /6: track 61.0 -> 88.2 mm
- net /7: track 59.1 -> 84.0 mm
- net /8: track 57.2 -> 79.7 mm
- net /9: track 55.2 -> 75.1 mm
- net /10: track 53.3 -> 71.3 mm
- net /11: track 50.8 -> 66.1 mm
- net /13: track 61.1 -> 75.1 mm, vias 2 -> 1
- net /12: track 60.6 -> 70.5 mm
- net /A4: track 69.4 -> 71.0 mm
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
Commit message: h2xS v2 in work
Routing:
- net GND: track 47.5 -> 168.3 mm, vias 0 -> 2
- net /A4: track 71.0 -> 108.7 mm
- net /A5: track 72.9 -> 107.3 mm
- net (no net): track 5.40 -> 16.1 mm

Commit message: h2xS v2 ready
Routing:
- net (no net): track 16.1 -> 21.5 mm
- net /A5: track 107.3 -> 106.8 mm
Other:
- board text added: "+5V"
- board text added: "D"
Changed lines of the file:
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@@
   (general
     (thickness 1.6)
-    (drawings 66)
-    (tracks 200)
+    (drawings 71)
+    (tracks 204)
     (zones 0)
     (modules 19)
@@
   )
   (setup
-    (last_trace_width 0.25)
+    (last_trace_width 0.8)
     (user_trace_width 0.5)
     (user_trace_width 0.6)
@@
     )
   )
+  (gr_line (start 137.4775 31.4325) (end 138.43 28) (layer F.SilkS) (width 0.12))
+  (gr_text Gnd (at 146.3675 29.5275) (layer F.SilkS)
+    (effects (font (size 1 1) (thickness 0.15)))
+  )
+  (gr_text +5V (at 143.1925 29.5275) (layer F.SilkS)
+    (effects (font (size 1 1) (thickness 0.15)))
+  )
+  (gr_text D (at 140.97 29.5275) (layer F.SilkS)
+    (effects (font (size 1 1) (thickness 0.15)))
+  )
+  (gr_text Vcc (at 60.325 34.925) (layer F.SilkS)
+    (effects (font (size 1 1) (thickness 0.15)))
+  )
+  (gr_text Gnd (at 60.325 32.385) (layer F.SilkS)
+    (effects (font (size 1 1) (thickness 0.15)))
+  )
   (gr_text 11 (at 128.27 61.2775) (layer F.Cu)
     (effects (font (size 1.5 1.5) (thickness 0.3)))
@@
     (effects (font (size 1.5 1.5) (thickness 0.3)))
   )
-  (gr_line (start 135.89 35.2425) (end 138.43 28) (layer F.SilkS) (width 0.12))
   (gr_text 2 (at 105.41 60.96 270) (layer F.SilkS)
     (effects (font (size 1 1) (thickness 0.15)))
@@
     (effects (font (size 1 1) (thickness 0.15)))
   )
-  (gr_text I2C (at 131.445 33.9725) (layer F.SilkS)
-    (effects (font (size 1 1) (thickness 0.15)))
-  )
-  (gr_line (start 127.635 39.0525) (end 127.635 35.2425) (layer F.SilkS) (width 0.12))
-  (gr_line (start 135.89 39.0525) (end 127.635 39.0525) (layer F.SilkS) (width 0.12))
-  (gr_line (start 135.89 35.2425) (end 135.89 39.0525) (layer F.SilkS) (width 0.12))
-  (gr_line (start 127.635 35.2425) (end 135.89 35.2425) (layer F.SilkS) (width 0.12))
-  (gr_text Gnd (at 134.62 37.1475 90) (layer F.SilkS)
-    (effects (font (size 1 1) (thickness 0.15)))
-  )
-  (gr_text Vcc (at 132.715 37.1475 90) (layer F.SilkS)
-    (effects (font (size 1 1) (thickness 0.15)))
-  )
-  (gr_text SCL (at 128.905 37.1475 90) (layer F.SilkS)
-    (effects (font (size 1 1) (thickness 0.15)))
-  )
-  (gr_text SDA (at 130.81 37.1475 90) (layer F.SilkS)
+  (gr_text I2C (at 133.985 30.1625) (layer F.SilkS)
+    (effects (font (size 1 1) (thickness 0.15)))
+  )
+  (gr_line (start 130.175 35.2425) (end 130.175 31.4325) (layer F.SilkS) (width 0.12))
+  (gr_line (start 138.43 35.2425) (end 130.175 35.2425) (layer F.SilkS) (width 0.12))
+  (gr_line (start 138.43 31.4325) (end 138.43 35.2425) (layer F.SilkS) (width 0.12))
+  (gr_line (start 130.175 31.4325) (end 138.43 31.4325) (layer F.SilkS) (width 0.12))
+  (gr_text Gnd (at 137.16 33.3375 90) (layer F.SilkS)
+    (effects (font (size 1 1) (thickness 0.15)))
+  )
+  (gr_text Vcc (at 135.255 33.3375 90) (layer F.SilkS)
+    (effects (font (size 1 1) (thickness 0.15)))
+  )
+  (gr_text SCL (at 131.445 33.3375 90) (layer F.SilkS)
+    (effects (font (size 1 1) (thickness 0.15)))
+  )
+  (gr_text SDA (at 133.35 33.3375 90) (layer F.SilkS)
     (effects (font (size 1 1) (thickness 0.15)))
   )
@@
   (segment (start 105.41 22.225) (end 105.41 23.495) (width 0.25) (layer F.Cu) (net 0))
   (segment (start 105.41 22.86) (end 106.9975 22.86) (width 0.25) (layer F.Cu) (net 0))
-  (segment (start 105.41 39.0525) (end 105.41 39.0525) (width 0.6) (layer F.Cu) (net 10))
+  (segment (start 53.975 32.385) (end 55.5625 32.385) (width 0.25) (layer F.Cu) (net 0))
+  (segment (start 53.975 31.75) (end 53.975 33.02) (width 0.25) (layer F.Cu) (net 0))
+  (segment (start 54.61 35.56) (end 54.61 34.33001) (width 0.25) (layer F.Cu) (net 0))
+  (segment (start 53.975 34.925) (end 55.245 34.925) (width 0.25) (layer F.Cu) (net 0))
   (segment (start 128.27 29.21) (end 128.27 29.21) (width 0.6) (layer F.Cu) (net 1))
   (segment (start 57.15 34.925) (end 62.865 34.925) (width 0.8) (layer B.Cu) (net 1))
@@
   (segment (start 107.95 22.86) (end 107.95 25.4) (width 0.6) (layer B.Cu) (net 9))
   (segment (start 108.64499 22.16501) (end 107.95 22.86) (width 0.6) (layer B.Cu) (net 9))
-  (segment (start 138.05251 22.16501) (end 108.64499 22.16501) (width 0.6) (layer B.Cu) (net 9))
-  (segment (start 138.43 23.495) (end 138.43 22.5425) (width 0.6) (layer B.Cu) (net 9))
-  (segment (start 138.43 22.5425) (end 138.05251 22.16501) (width 0.6) (layer B.Cu) (net 9))
+  (segment (start 136.24751 22.16501) (end 108.64499 22.16501) (width 0.6) (layer B.Cu) (net 9))
+  (segment (start 138.43 23.495) (end 137.4775 23.495) (width 0.6) (layer B.Cu) (net 9))
+  (segment (start 137.4775 23.495) (end 136.24751 22.16501) (width 0.6) (layer B.Cu) (net 9))
+  (segment (start 105.41 39.0525) (end 105.41 39.0525) (width 0.6) (layer F.Cu) (net 10))
   (segment (start 62.23 31.115) (end 62.23 25.4) (width 0.8) (layer B.Cu) (net 10))
   (segment (start 57.15 32.385) (end 60.96 32.385) (width 0.8) (layer B.Cu) (net 10))
