File: modules/R-2R/R-2R.sch (KiCad schematic (older format))
At the start: 25 parts, among them J1 Conn_01x10_Male, J2 Conn_01x10_Male, J3 Conn_01x01_Male, U1 74LS573

Commit message: R-2R, polishing
Parts:
- added J4: Conn_01x01_Male, Connector_PinHeader_2.54mm:PinHeader_1x01_P2.54mm_Vertical, symbol Connector:Conn_01x01_Male
Connections:
- net GND: now also J4.1 (Pin_1)
Changed lines of the file:
@@
 NoConn ~ 1750 2800
 NoConn ~ 3000 2900
+$Comp
+L Connector:Conn_01x01_Male J4
+U 1 1 5EA7598C
+P 5450 1600
+F 0 "J4" V 5600 1550 50  0000 R CNN
+F 1 "Conn_01x01_Male" V 5475 1550 50  0000 R CNN
+F 2 "Connector_PinHeader_2.54mm:PinHeader_1x01_P2.54mm_Vertical" H 5450 1600 50  0001 C CNN
+F 3 "~" H 5450 1600 50  0001 C CNN
+	1    5450 1600
+	0    -1   1    0
+$EndComp
+$Comp
+L power:GND #PWR0104
+U 1 1 5EA7649F
+P 5450 1800
+F 0 "#PWR0104" H 5450 1550 50  0001 C CNN
+F 1 "GND" H 5455 1627 50  0000 C CNN
+F 2 "" H 5450 1800 50  0001 C CNN
+F 3 "" H 5450 1800 50  0001 C CNN
+	1    5450 1800
+	1    0    0    -1
+$EndComp
 $EndSCHEMATC
