File: modules/L293v2/L293.sch (KiCad schematic (older format))
At the start: 38 parts, among them J1 2, J10 11, J11 12, J12 13, J13 A0, J14 A1, J15 A2, J16 A3, J17 A4, J18 A5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

Commit message: Motor shield polishing
Parts:
- added C3: 0.1uF, Capacitor_SMD:C_0805_2012Metric_Pad1.15x1.40mm_HandSolder, symbol Device:C
- added J24, J25: Conn_01x01_Male, Connector_PinHeader_2.54mm:PinHeader_1x01_P2.54mm_Vertical, symbol Connector:Conn_01x01_Male
- added R3: 10k, Resistor_SMD:R_0805_2012Metric_Pad1.15x1.40mm_HandSolder, symbol Device:R
- added R4: 50k, Resistor_SMD:R_0805_2012Metric_Pad1.15x1.40mm_HandSolder, symbol Device:R
Connections:
- net GND: now also C3.1, R3.1
- net M1+: now also J8.1 (Pin_1), U1.13 (D3); no longer J7.1 (Pin_1), U1.12 (D2)
- net M1-: now also J7.1 (Pin_1), U1.12 (D2); no longer J8.1 (Pin_1), U1.13 (D3)
- net at C2.2, C4.1, C5.1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: now also R4.1
- net at R2.2, U1.1 (~Mr): now also J24.1 (Pin_1)
- new net: C3.2, J25.1 (Pin_1), R3.2, R4.2
Other:
- note added: "Check battery voltage here!"
- note added: "Reset"
Changed lines of the file:
@@
 P 4175 1800
 F 0 "#FLG0103" H 4175 1875 50  0001 C CNN
-F 1 "PWR_FLAG" H 4175 1973 50  0000 C CNN
+F 1 "PWR_FLAG" H 4400 1925 50  0000 C CNN
 F 2 "" H 4175 1800 50  0001 C CNN
 F 3 "~" H 4175 1800 50  0001 C CNN
@@
 Text Label 1475 2950 0    50   ~ 0
 PWM2
+Text Label 1325 3550 0    50   ~ 0
+M1+
 Text Label 1325 3400 0    50   ~ 0
-M1+
-Text Label 1350 3550 0    50   ~ 0
 M1-
 Text Label 1375 3700 0    50   ~ 0
@@
 NoConn ~ 3000 3300
 $Comp
-L power:VCC #PWR08
-U 1 1 5FAF8DE2
-P 4925 5400
-F 0 "#PWR08" H 4925 5250 50  0001 C CNN
-F 1 "VCC" H 4940 5573 50  0000 C CNN
-F 2 "" H 4925 5400 50  0001 C CNN
-F 3 "" H 4925 5400 50  0001 C CNN
-	1    4925 5400
-	1    0    0    -1
-$EndComp
-$Comp
 L Device:R R2
 U 1 1 5FB01962
@@
 	1950 2600 2000 2600
 $Comp
-L power:VCC #PWR?
+L power:VCC #PWR09
 U 1 1 5FAF2DDD
 P 2500 3700
-F 0 "#PWR?" H 2500 3550 50  0001 C CNN
+F 0 "#PWR09" H 2500 3550 50  0001 C CNN
 F 1 "VCC" H 2515 3873 50  0000 C CNN
 F 2 "" H 2500 3700 50  0001 C CNN
@@
 	-1   0    0    1
 $EndComp
+$Comp
+L Connector:Conn_01x01_Male J24
+U 1 1 5FADBB27
+P 1800 2500
+F 0 "J24" H 1800 2575 50  0000 C CNN
+F 1 "Conn_01x01_Male" H 1700 2450 50  0000 C CNN
+F 2 "Connector_PinHeader_2.54mm:PinHeader_1x01_P2.54mm_Vertical" H 1800 2500 50  0001 C CNN
+F 3 "~" H 1800 2500 50  0001 C CNN
+	1    1800 2500
+	1    0    0    -1
+$EndComp
+Connection ~ 2000 2500
+$Comp
+L Connector:Conn_01x01_Male J25
+U 1 1 5FADCDAD
+P 3750 1500
+F 0 "J25" H 3750 1575 50  0000 C CNN
+F 1 "Conn_01x01_Male" H 4350 1550 50  0000 C CNN
+F 2 "Connector_PinHeader_2.54mm:PinHeader_1x01_P2.54mm_Vertical" H 3750 1500 50  0001 C CNN
+F 3 "~" H 3750 1500 50  0001 C CNN
+	1    3750 1500
+	1    0    0    1
+$EndComp
+$Comp
+L Device:R R4
+U 1 1 5FADEC8D
+P 3950 1650
+F 0 "R4" H 4100 1675 50  0000 R CNN
+F 1 "50k" V 3950 1725 50  0000 R CNN
+F 2 "Resistor_SMD:R_0805_2012Metric_Pad1.15x1.40mm_HandSolder" V 3880 1650 50  0001 C CNN
+F 3 "~" H 3950 1650 50  0001 C CNN
+	1    3950 1650
+	1    0    0    1
+$EndComp
+$Comp
+L Device:R R3
+U 1 1 5FADFB3B
+P 3950 1350
+F 0 "R3" H 4000 1375 50  0000 L CNN
+F 1 "10k" V 3950 1300 50  0000 L CNN
+F 2 "Resistor_SMD:R_0805_2012Metric_Pad1.15x1.40mm_HandSolder" V 3880 1350 50  0001 C CNN
+F 3 "~" H 3950 1350 50  0001 C CNN
+	1    3950 1350
+	1    0    0    -1
+$EndComp
+Connection ~ 3950 1500
+$Comp
+L power:GND #PWR010
+U 1 1 5FAE7967
+P 3950 1200
+F 0 "#PWR010" H 3950 950 50  0001 C CNN
+F 1 "GND" H 3955 1027 50  0000 C CNN
+F 2 "" H 3950 1200 50  0001 C CNN
+F 3 "" H 3950 1200 50  0001 C CNN
+	1    3950 1200
+	-1   0    0    1
+$EndComp
+$Comp
+L Device:C C3
+U 1 1 5FAEF0CB
+P 4200 1350
+F 0 "C3" H 4315 1396 50  0000 L CNN
+F 1 "0.1uF" H 4315 1305 50  0000 L CNN
+F 2 "Capacitor_SMD:C_0805_2012Metric_Pad1.15x1.40mm_HandSolder" H 4238 1200 50  0001 C CNN
+F 3 "~" H 4200 1350 50  0001 C CNN
+	1    4200 1350
+	1    0    0    -1
+$EndComp
+$Comp
+L power:GND #PWR011
+U 1 1 5FAEFA4D
+P 4200 1200
+F 0 "#PWR011" H 4200 950 50  0001 C CNN
+F 1 "GND" H 4205 1027 50  0000 C CNN
+F 2 "" H 4200 1200 50  0001 C CNN
+F 3 "" H 4200 1200 50  0001 C CNN
+	1    4200 1200
+	-1   0    0    1
+$EndComp
+Wire Wire Line
+	3950 1500 4200 1500
+Text Notes 3800 1475 1    50   ~ 0
+Check battery voltage here!
+Text Notes 1850 2375 1    50   ~ 0
+Reset
 $EndSCHEMATC

Commit message: L293. Reverse polarity protection is added.
Parts:
- added Q1: IRLML5203, Package_TO_SOT_SMD:SOT-23, symbol Transistor_FET:IRLML5203
Connections:
- net GND: now also Q1.1 (G)
- net at C2.2, C4.1, C5.1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: now also Q1.2 (S); no longer J21.1 (Pin_1)
- new net: J21.1 (Pin_1), Q1.3 (D)
Other:
- note added: "Reverse\npolarity\nprotection"
- moved on the sheet: J21
Changed lines of the file:
@@
 L Connector:Screw_Terminal_01x02 J21
 U 1 1 5E5027C6
-P 4575 1800
-F 0 "J21" H 4655 1792 50  0000 L CNN
-F 1 "Pwr" H 4655 1701 50  0000 L CNN
-F 2 "TerminalBlock:TerminalBlock_bornier-2_P5.08mm" H 4575 1800 50  0001 C CNN
-F 3 "~" H 4575 1800 50  0001 C CNN
-	1    4575 1800
+P 5150 1800
+F 0 "J21" H 5230 1792 50  0000 L CNN
+F 1 "Pwr" H 5230 1701 50  0000 L CNN
+F 2 "TerminalBlock:TerminalBlock_bornier-2_P5.08mm" H 5150 1800 50  0001 C CNN
+F 3 "~" H 5150 1800 50  0001 C CNN
+	1    5150 1800
 	1    0    0    -1
 $EndComp
@@
 Connection ~ 4175 1800
 Wire Wire Line
-	4175 1800 4375 1800
-Wire Wire Line
 	4175 2100 4275 2100
-Wire Wire Line
-	4375 2100 4275 2100
-Wire Wire Line
-	4375 1900 4375 2100
 Connection ~ 4275 2100
 $Comp
@@
 P 3750 1500
 F 0 "J25" H 3750 1575 50  0000 C CNN
-F 1 "Conn_01x01_Male" H 4350 1550 50  0000 C CNN
+F 1 "Conn_01x01_Male" V 3675 1025 50  0000 C CNN
 F 2 "Connector_PinHeader_2.54mm:PinHeader_1x01_P2.54mm_Vertical" H 3750 1500 50  0001 C CNN
 F 3 "~" H 3750 1500 50  0001 C CNN
@@
 Text Notes 1850 2375 1    50   ~ 0
 Reset
+$Comp
+L Transistor_FET:IRLML5203 Q1
+U 1 1 5FC35DF4
+P 4750 1900
+F 0 "Q1" V 4650 1975 50  0000 C CNN
+F 1 "IRLML5203" V 4975 2025 50  0000 C CNN
+F 2 "Package_TO_SOT_SMD:SOT-23" H 4950 1825 50  0001 L CIN
+F 3 "https://www.infineon.com/dgdl/irlml5203pbf.pdf?fileId=5546d462533600a40153566868da261d" H 4750 1900 50  0001 L CNN
+	1    4750 1900
+	0    1    -1   0
+$EndComp
+Wire Wire Line
+	4175 1800 4550 1800
+Wire Wire Line
+	4275 2100 4750 2100
+Wire Wire Line
+	4750 2100 4950 2100
+Wire Wire Line
+	4950 2100 4950 1900
+Connection ~ 4750 2100
+Text Notes 4650 1600 0    50   ~ 0
+Reverse\npolarity\nprotection
 $EndSCHEMATC
