File: modules/SmdKbd/SmdKbd.sch (KiCad schematic (older format))
At the start: 28 parts, among them J1 Conn_01x10_Male, J2 Conn_01x10_Male, SW1 SW_Push, SW10 SW_Push, SW11 SW_Push, SW12 SW_Push, SW13 SW_Push, SW14 SW_Push, SW15 SW_Push, SW16 SW_Push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

Commit message: SmdKbd in work
Connections:
- wire segments 67 -> 81
Changed lines of the file:
@@
 	0    -1   -1   0
 $EndComp
+Wire Wire Line
+	4900 2500 4900 3000
+Wire Wire Line
+	4900 3000 4900 3500
+Connection ~ 4900 3000
+Wire Wire Line
+	4900 3500 4900 4000
+Connection ~ 4900 3500
+Wire Wire Line
+	5650 2500 5650 3000
+Wire Wire Line
+	5650 3000 5650 3500
+Connection ~ 5650 3000
+Wire Wire Line
+	5650 3500 5650 4000
+Connection ~ 5650 3500
+Wire Wire Line
+	7150 2500 7150 3000
+Wire Wire Line
+	7150 3000 7150 3500
+Connection ~ 7150 3000
+Wire Wire Line
+	7150 3500 7150 4000
+Connection ~ 7150 3500
+Wire Wire Line
+	7900 2500 7900 3000
+Wire Wire Line
+	7900 3000 7900 3500
+Connection ~ 7900 3000
+Wire Wire Line
+	7900 3500 7900 4000
+Connection ~ 7900 3500
+Wire Wire Line
+	4900 2500 5000 2500
+Connection ~ 4900 2500
+Wire Wire Line
+	5650 2500 5750 2500
+Connection ~ 5650 2500
+Text Label 5000 2500 0    50   ~ 0
+A3
 $EndSCHEMATC
